Commit message: in work

File: aster_description/urdf/aster.xacro (robot description, xacro)
@@ -8,6 +8,8 @@
                 <mesh filename="package://aster_description/meshes/ownStls/standBase.stl" scale="0.001 0.001 0.001"/>
             </geometry>
+            <material name="white"/>
         </visual>
     </link>
+    <!-- Base-->
     <link name="base_holder_link">
         <visual>
@@ -16,4 +18,5 @@
                 <mesh filename="package://aster_description/meshes/subStuff/RohrHalter_v2.stl" scale="0.001 0.001 0.001"/>
             </geometry>
+            <material name="white"/>
         </visual>
     </link>
@@ -24,6 +27,60 @@
                 <mesh filename="package://aster_description/meshes/Spine_Connector.stl" scale="0.001 0.001 0.001"/>
             </geometry>
+            <material name="white"/>
         </visual>
     </link>
+    <link name="chest_link">
+        <visual>
+            <origin xyz="0.0 0.0 -0.012" rpy="0.0 0.0 0.0"/>
+            <geometry>
+                <mesh filename="package://aster_description/meshes/Chest.stl" scale="0.001 0.001 0.001"/>
+            </geometry>
+            <material name="blue"/>
+        </visual>
+    </link>
+    <link name="backbone_link">
+        <visual>
+            <origin xyz="-0.003 0.0 -0.085" rpy="0.0 0.0 0.0"/>
+            <geometry>
+                <mesh filename="package://aster_description/meshes/Spine.stl" scale="0.001 0.001 0.001"/>
+            </geometry>
+            <material name="blue"/>
+        </visual>
+    </link>
+    <link name="hip_link">
+        <visual>
+            <origin xyz="-0.005 0.0 0.003" rpy="0.0 0.0 0.0"/>
+            <geometry>
+                <mesh filename="package://aster_description/meshes/Hips.stl" scale="0.001 0.001 0.001"/>
+            </geometry>
+            <material name="blue"/>
+        </visual>
+    </link>
+   <!-- Head-->
+    <link name="neck_link">
+        <visual>
+            <origin xyz="0.0 0.0 -0.012" rpy="0.0 0.0 0.0"/>
+            <geometry>
+                <mesh filename="package://aster_description/meshes/Head_Neck.stl" scale="0.001 0.001 0.001"/>
+            </geometry>
+            <material name="blue"/>
+        </visual>
+    </link>
+    <link name="head_link">
+        <visual>
+            <origin xyz="0.0 0.0 -0.012" rpy="0.0 0.0 0.0"/>
+            <geometry>
+                <mesh filename="package://aster_description/meshes/Head_Back.stl" scale="0.001 0.001 0.001"/>
+            </geometry>
+            <material name="white"/>
+        </visual>
+    </link>
+    <!-- Right Arm-->
+    <!-- Right Gripper-->
+    <!-- Left Arm-->
+    <!-- Left Gripper-->
+    <!-- Right Leg-->
+    <!-- Left Leg-->
+    <!-- Base Virtual Joints-->
     <joint name="virtual_1_joint" type="fixed">
         <parent link="world"/>
@@ -39,5 +96,41 @@
         <parent link="base_holder_link"/>
         <child link="chest_bone_link"/>
-        <origin xyz="0.035 0.0 0.01" rpy="0.0 0.0 0.0"/>
+        <origin xyz="0.042 0.0 0.015" rpy="0.0 0.0 0.0"/>
     </joint>
+    <joint name="virtual_4_joint" type="fixed">
+        <parent link="chest_bone_link"/>
+        <child link="chest_link"/>
+        <origin xyz="0 0 0" rpy="0.0 0.0 0.0"/>
+    </joint>
+    <joint name="virtual_5_joint" type="fixed">
+        <parent link="chest_bone_link"/>
+        <child link="backbone_link"/>
+        <origin xyz="0 0 0" rpy="0.0 0.0 0.0"/>
+    </joint>
+    <joint name="virtual_6_joint" type="fixed">
+        <parent link="backbone_link"/>
+        <child link="hip_link"/>
+        <origin xyz="0 0 -0.2" rpy="0.0 0.0 0.0"/>
+    </joint>
+     <!--Head Joints-->
+    <joint name="joint_1" type="revolute">
+        <parent link="chest_link"/>
+        <child link="neck_link"/>
+        <axis xyz="0 0 1 "/>
+        <limit lower="-1.57" upper="1.57" velocity="50.0" effort="1000.0"/>
+        <origin xyz="0 0 0.1" rpy="0 0 0"/>
+    </joint>
+    <joint name="joint_2" type="revolute">
+        <parent link="neck_link"/>
+        <child link="head_link"/>
+        <axis xyz="0 1 0"/>
+        <limit lower="-0.5" upper="0.3" velocity="50.0" effort="1000.0"/>
+        <origin xyz="0 0 0.01" rpy="0 0 0"/>
+    </joint>
+    <!-- Right Arm Joints-->
+    <!-- Right Gripper Joints-->
+    <!-- Left Arm Joints-->
+    <!-- Left Gripper Joints-->
+    <!-- Right Leg Joints-->
+    <!-- Left Leg Joints-->
 </robot>

Commit message: upper body is ready without gripper

File: aster_description/urdf/aster.xacro (robot description, xacro)
@@ -77,6 +77,80 @@
     </link>
     <!-- Right Arm-->
+    <link name="shoulder_rh_link">
+        <visual>
+            <origin xyz="-0.01 -0.018 -0.023" rpy="0.0 0.0 0.0"/>
+            <geometry>
+                <mesh filename="package://aster_description/meshes/Rigth_Arm_Shoulder_Connector.stl" scale="0.001 0.001 0.001"/>
+            </geometry>
+            <material name="white"/>
+        </visual>
+    </link>
+    <link name="sh_rh_lift_link">
+        <visual>
+            <origin xyz="0 0.108 -0.6625" rpy="0.0 0.0 0.0"/>
+            <geometry>
+                <mesh filename="package://aster_description/meshes/Right_Arm_Shoulder.stl" scale="0.001 0.001 0.001"/>
+            </geometry>
+            <material name="white"/>
+        </visual>
+    </link>
+    <link name="sh_rh_rotate_link">
+        <visual>
+            <origin xyz="0 0.108 0.51" rpy="3.1415 0.0 3.1415"/>
+            <geometry>
+                <mesh filename="package://aster_description/meshes/Right_Arm_Upper.stl" scale="0.001 0.001 0.001"/>
+            </geometry>
+            <material name="white"/>
+        </visual>
+    </link>
+    <link name="elbow_rh_link">
+        <visual>
+            <origin xyz="-0.01 0.1075 -0.498" rpy="0 0 0"/>
+            <geometry>
+                <mesh filename="package://aster_description/meshes/Right_Arm_Lower.stl" scale="0.001 0.001 0.001"/>
+            </geometry>
+            <material name="white"/>
+        </visual>
+    </link>
+    <link name="rh_rotate_link" />
     <!-- Right Gripper-->
     <!-- Left Arm-->
+    <link name="shoulder_lh_link">
+        <visual>
+            <origin xyz="-0.01 0.018 -0.023" rpy="0.0 0.0 0.0"/>
+            <geometry>
+                <mesh filename="package://aster_description/meshes/Left_Arm_Shoulder_Connector.stl" scale="0.001 0.001 0.001"/>
+            </geometry>
+            <material name="white"/>
+        </visual>
+    </link>
+    <link name="sh_lh_lift_link">
+        <visual>
+            <origin xyz="0 0 -0.036" rpy="0.0 0.0 0.0"/>
+            <geometry>
+                <mesh filename="package://aster_description/meshes/Left_Arm_Shoulder.stl" scale="0.001 0.001 0.001"/>
+            </geometry>
+            <material name="white"/>
+        </visual>
+    </link>
+    <link name="sh_lh_rotate_link">
+        <visual>
+            <origin xyz="0 0 -0.005" rpy="3.1415 0.0 3.1415"/>
+            <geometry>
+                <mesh filename="package://aster_description/meshes/Left_Arm_Upper.stl" scale="0.001 0.001 0.001"/>
+            </geometry>
+            <material name="white"/>
+        </visual>
+    </link>
+    <link name="elbow_lh_link">
+        <visual>
+            <origin xyz="-0.06 0.002 -0.008" rpy="0 0 0"/>
+            <geometry>
+                <mesh filename="package://aster_description/meshes/Left_Arm_Lower.stl" scale="0.001 0.001 0.001"/>
+            </geometry>
+            <material name="white"/>
+        </visual>
+    </link>
+    <link name="lh_rotate_link" />
     <!-- Left Gripper-->
     <!-- Right Leg-->
@@ -129,6 +203,76 @@
     </joint>
     <!-- Right Arm Joints-->
+    <joint name="joint_3" type="revolute">
+        <parent link="chest_link"/>
+        <child link="shoulder_rh_link"/>
+        <axis xyz="0 1 0"/>
+        <limit lower="-1.57" upper="1.57" velocity="50.0" effort="1000.0"/>
+        <origin xyz="0.0 -0.085 0.05" rpy="0 0 0"/>
+    </joint>
+    <joint name="joint_4" type="revolute">
+        <parent link="shoulder_rh_link"/>
+        <child link="sh_rh_lift_link"/>
+        <axis xyz="1 0 0"/>
+        <limit lower="-1.57" upper="0" velocity="50.0" effort="1000.0"/>
+        <origin xyz="-0.008 -0.027 0" rpy="0 0 0"/>
+    </joint>
+    <joint name="joint_5" type="revolute">
+        <parent link="sh_rh_lift_link"/>
+        <child link="sh_rh_rotate_link"/>
+        <axis xyz="0 0 1"/>
+        <limit lower="-1.57" upper="1.57" velocity="50.0" effort="1000.0"/>
+        <origin xyz="0 0 -0.04" rpy="0 0 0"/>
+    </joint>
+    <joint name="joint_6" type="revolute">
+        <parent link="sh_rh_rotate_link"/>
+        <child link="elbow_rh_link"/>
+        <axis xyz="0 1 0"/>
+        <limit lower="-1.57" upper="0" velocity="50.0" effort="1000.0"/>
+        <origin xyz="0 0 -0.13" rpy="0 0 0"/>
+    </joint>
+    <joint name="joint_7" type="revolute">
+        <parent link="elbow_rh_link"/>
+        <child link="rh_rotate_link"/>
+        <axis xyz="0 0 1"/>
+        <limit lower="0" upper="1.57" velocity="50.0" effort="1000.0"/>
+        <origin xyz="0 -0.01 -0.13" rpy="0 0 0"/>
+    </joint>
     <!-- Right Gripper Joints-->
     <!-- Left Arm Joints-->
+    <joint name="joint_9" type="revolute">
+        <parent link="chest_link"/>
+        <child link="shoulder_lh_link"/>
+        <axis xyz="0 1 0"/>
+        <limit lower="-1.57" upper="1.57" velocity="50.0" effort="1000.0"/>
+        <origin xyz="0.0 0.085 0.05" rpy="0 0 0"/>
+    </joint>
+    <joint name="joint_10" type="revolute">
+        <parent link="shoulder_lh_link"/>
+        <child link="sh_lh_lift_link"/>
+        <axis xyz="1 0 0"/>
+        <limit lower="0" upper="1.57" velocity="50.0" effort="1000.0"/>
+        <origin xyz="-0.008 0.027 0" rpy="0 0 0"/>
+    </joint>
+    <joint name="joint_11" type="revolute">
+        <parent link="sh_lh_lift_link"/>
+        <child link="sh_lh_rotate_link"/>
+        <axis xyz="0 0 1"/>
+        <limit lower="-1.57" upper="1.57" velocity="50.0" effort="1000.0"/>
+        <origin xyz="0 0 -0.04" rpy="0 0 0"/>
+    </joint>
+    <joint name="joint_12" type="revolute">
+        <parent link="sh_lh_rotate_link"/>
+        <child link="elbow_lh_link"/>
+        <axis xyz="0 1 0"/>
+        <limit lower="-1.57" upper="0" velocity="50.0" effort="1000.0"/>
+        <origin xyz="0 0 -0.13" rpy="0 0 0"/>
+    </joint>
+    <joint name="joint_13" type="revolute">
+        <parent link="elbow_lh_link"/>
+        <child link="lh_rotate_link"/>
+        <axis xyz="0 0 1"/>
+        <limit lower="-1.57" upper="0" velocity="50.0" effort="1000.0"/>
+        <origin xyz="0 0.015 -0.13" rpy="0 0 0"/>
+    </joint>
     <!-- Left Gripper Joints-->
     <!-- Right Leg Joints-->

Commit message: gripper ready for rviz2

File: aster_description/urdf/aster.xacro (robot description, xacro)
@@ -113,6 +113,41 @@
         </visual>
     </link>
-    <link name="rh_rotate_link" />
     <!-- Right Gripper-->
+    <link name="rh_rotate_link" >
+        <visual>
+            <origin xyz="-0.02 0 -0.03" rpy="-1.57 0 -1.57"/>
+            <geometry>
+                <mesh filename="package://aster_description/meshes/Greifer/files/Robotic_Arm_Palm.stl" scale="0.001 0.001 0.001"/>
+            </geometry>
+            <material name="white"/>
+        </visual>
+    </link>
+    <link name="rh_rotate_top_link" >
+        <visual>
+            <origin xyz="-0.004 0 -0.03" rpy="-1.57 0 -1.57"/>
+            <geometry>
+                <mesh filename="package://aster_description/meshes/Greifer/files/Robotic_Arm_Palm_Top.stl" scale="0.001 0.001 0.001"/>
+            </geometry>
+            <material name="white"/>
+        </visual>
+    </link>
+    <link name="rh_gripper1_link" >
+        <visual>
+            <origin xyz="-0.005 0.016 -0.008" rpy="-1.57 0 -1.57"/>
+            <geometry>
+                <mesh filename="package://aster_description/meshes/Greifer/files/Robotic_Arm_Finger.stl" scale="0.001 0.001 0.001"/>
+            </geometry>
+            <material name="white"/>
+        </visual>
+    </link>
+    <link name="rh_gripper2_link" >
+        <visual>
+            <origin xyz="0.007 -0.016 -0.008" rpy="-1.57 0 1.57"/>
+            <geometry>
+                <mesh filename="package://aster_description/meshes/Greifer/files/Robotic_Arm_Finger.stl" scale="0.001 0.001 0.001"/>
+            </geometry>
+            <material name="white"/>
+        </visual>
+    </link>
     <!-- Left Arm-->
     <link name="shoulder_lh_link">
@@ -152,8 +187,44 @@
         </visual>
     </link>
-    <link name="lh_rotate_link" />
     <!-- Left Gripper-->
+    <link name="lh_rotate_link" >
+        <visual>
+            <origin xyz="-0.02 0 -0.03" rpy="-1.57 0 -1.57"/>
+            <geometry>
+                <mesh filename="package://aster_description/meshes/Greifer/files/Robotic_Arm_Palm.stl" scale="0.001 0.001 0.001"/>
+            </geometry>
+            <material name="white"/>
+        </visual>
+    </link>
+    <link name="lh_rotate_top_link" >
+        <visual>
+            <origin xyz="-0.004 0 -0.03" rpy="-1.57 0 -1.57"/>
+            <geometry>
+                <mesh filename="package://aster_description/meshes/Greifer/files/Robotic_Arm_Palm_Top.stl" scale="0.001 0.001 0.001"/>
+            </geometry>
+            <material name="white"/>
+        </visual>
+    </link>
+    <link name="lh_gripper1_link" >
+        <visual>
+            <origin xyz="-0.005 0.016 -0.008" rpy="-1.57 0 -1.57"/>
+            <geometry>
+                <mesh filename="package://aster_description/meshes/Greifer/files/Robotic_Arm_Finger.stl" scale="0.001 0.001 0.001"/>
+            </geometry>
+            <material name="white"/>
+        </visual>
+    </link>
+    <link name="lh_gripper2_link" >
+        <visual>
+            <origin xyz="0.007 -0.016 -0.008" rpy="-1.57 0 1.57"/>
+            <geometry>
+                <mesh filename="package://aster_description/meshes/Greifer/files/Robotic_Arm_Finger.stl" scale="0.001 0.001 0.001"/>
+            </geometry>
+            <material name="white"/>
+        </visual>
+    </link>
     <!-- Right Leg-->
     <!-- Left Leg-->
+                    <!-- ######  JOINTS  ######-->
     <!-- Base Virtual Joints-->
     <joint name="virtual_1_joint" type="fixed">
@@ -231,4 +302,5 @@
         <origin xyz="0 0 -0.13" rpy="0 0 0"/>
     </joint>
+    <!-- Right Gripper Joints-->
     <joint name="joint_7" type="revolute">
         <parent link="elbow_rh_link"/>
@@ -238,5 +310,24 @@
         <origin xyz="0 -0.01 -0.13" rpy="0 0 0"/>
     </joint>
-    <!-- Right Gripper Joints-->
+    <joint name="virtual_7_joint" type="fixed">
+        <parent link="rh_rotate_link"/>
+        <child link="rh_rotate_top_link"/>
+        <origin xyz="0.0 0.0 0.0" rpy="0.0 0.0 0.0"/>
+    </joint>
+    <joint name="joint_8" type="revolute">
+        <parent link="rh_rotate_link"/>
+        <child link="rh_gripper1_link"/>
+        <axis xyz="1 0 0"/>
+        <limit lower="-0.76" upper="0" velocity="50.0" effort="1000.0"/>
+        <origin xyz="-0.015 -0.02 -0.048" rpy="0 0 0"/>
+    </joint>
+    <joint name="joint_8_m" type="revolute">
+        <mimic joint="joint_8" multiplier="-1"/>
+        <parent link="rh_rotate_link"/>
+        <child link="rh_gripper2_link"/>
+        <axis xyz="1 0 0"/>
+        <limit lower="0" upper="0.76" velocity="50.0" effort="1000.0"/>
+        <origin xyz="-0.015 0.02 -0.048" rpy="0 0 0"/>
+    </joint>
     <!-- Left Arm Joints-->
     <joint name="joint_9" type="revolute">
@@ -268,4 +359,5 @@
         <origin xyz="0 0 -0.13" rpy="0 0 0"/>
     </joint>
+    <!-- Left Gripper Joints-->
     <joint name="joint_13" type="revolute">
         <parent link="elbow_lh_link"/>
@@ -275,5 +367,24 @@
         <origin xyz="0 0.015 -0.13" rpy="0 0 0"/>
     </joint>
-    <!-- Left Gripper Joints-->
+    <joint name="virtual_10_joint" type="fixed">
+        <parent link="lh_rotate_link"/>
+        <child link="lh_rotate_top_link"/>
+        <origin xyz="0.0 0.0 0.0" rpy="0.0 0.0 0.0"/>
+    </joint>
+    <joint name="joint_14" type="revolute">
+        <parent link="lh_rotate_link"/>
+        <child link="lh_gripper1_link"/>
+        <axis xyz="1 0 0"/>
+        <limit lower="-0.76" upper="0" velocity="50.0" effort="1000.0"/>
+        <origin xyz="-0.015 -0.02 -0.048" rpy="0 0 0"/>
+    </joint>
+    <joint name="joint_14_m" type="revolute">
+        <mimic joint="joint_14" multiplier="-1"/>
+        <parent link="lh_rotate_link"/>
+        <child link="lh_gripper2_link"/>
+        <axis xyz="1 0 0"/>
+        <limit lower="0" upper="0.76" velocity="50.0" effort="1000.0"/>
+        <origin xyz="-0.015 0.02 -0.048" rpy="0 0 0"/>
+    </joint>
     <!-- Right Leg Joints-->
     <!-- Left Leg Joints-->
