Commit message: upper body is ready in rviz2 with gripper and gipper_pads

File: aster_description/urdf/aster.xacro (robot description, xacro)
@@ -97,5 +97,5 @@
     <link name="sh_rh_rotate_link">
         <visual>
-            <origin xyz="0 0.108 0.51" rpy="3.1415 0.0 3.1415"/>
+            <origin xyz="0 0.108 0.51" rpy="${PI} 0 ${PI}"/>
             <geometry>
                 <mesh filename="package://aster_description/meshes/Right_Arm_Upper.stl" scale="0.001 0.001 0.001"/>
@@ -116,5 +116,5 @@
     <link name="rh_rotate_link" >
         <visual>
-            <origin xyz="-0.02 0 -0.03" rpy="-1.57 0 -1.57"/>
+            <origin xyz="-0.02 0 -0.03" rpy="${-PI/2} 0 ${-PI/2}"/>
             <geometry>
                 <mesh filename="package://aster_description/meshes/Greifer/files/Robotic_Arm_Palm.stl" scale="0.001 0.001 0.001"/>
@@ -125,5 +125,5 @@
     <link name="rh_rotate_top_link" >
         <visual>
-            <origin xyz="-0.004 0 -0.03" rpy="-1.57 0 -1.57"/>
+            <origin xyz="-0.004 0 -0.03" rpy="${-PI/2} 0 ${-PI/2}"/>
             <geometry>
                 <mesh filename="package://aster_description/meshes/Greifer/files/Robotic_Arm_Palm_Top.stl" scale="0.001 0.001 0.001"/>
@@ -134,5 +134,5 @@
     <link name="rh_gripper1_link" >
         <visual>
-            <origin xyz="-0.005 0.016 -0.008" rpy="-1.57 0 -1.57"/>
+            <origin xyz="-0.005 0.016 -0.008" rpy="${-PI/2} 0 ${-PI/2}"/>
             <geometry>
                 <mesh filename="package://aster_description/meshes/Greifer/files/Robotic_Arm_Finger.stl" scale="0.001 0.001 0.001"/>
@@ -143,9 +143,27 @@
     <link name="rh_gripper2_link" >
         <visual>
-            <origin xyz="0.007 -0.016 -0.008" rpy="-1.57 0 1.57"/>
+            <origin xyz="0.007 -0.016 -0.008" rpy="${-PI/2} 0 ${PI/2}"/>
             <geometry>
                 <mesh filename="package://aster_description/meshes/Greifer/files/Robotic_Arm_Finger.stl" scale="0.001 0.001 0.001"/>
             </geometry>
             <material name="white"/>
+        </visual>
+    </link>
+    <link name="rh_gripper1_pad_link" >
+        <visual>
+            <origin xyz="-0.004 -0.0015 -0.0017" rpy="0 ${PI/2} 0"/>
+            <geometry>
+                <mesh filename="package://aster_description/meshes/Greifer/files/Robotic_Arm_Finger_Pad.stl" scale="0.001 0.001 0.001"/>
+            </geometry>
+            <material name="blue"/>
+        </visual>
+    </link>
+    <link name="rh_gripper2_pad_link" >
+        <visual>
+            <origin xyz="0.005 0.0015 -0.0017" rpy="${PI} ${PI/2} 0"/>
+            <geometry>
+                <mesh filename="package://aster_description/meshes/Greifer/files/Robotic_Arm_Finger_Pad.stl" scale="0.001 0.001 0.001"/>
+            </geometry>
+            <material name="blue"/>
         </visual>
     </link>
@@ -171,5 +189,5 @@
     <link name="sh_lh_rotate_link">
         <visual>
-            <origin xyz="0 0 -0.005" rpy="3.1415 0.0 3.1415"/>
+            <origin xyz="0 0 -0.005" rpy="${PI} 0 ${PI}"/>
             <geometry>
                 <mesh filename="package://aster_description/meshes/Left_Arm_Upper.stl" scale="0.001 0.001 0.001"/>
@@ -190,5 +208,5 @@
     <link name="lh_rotate_link" >
         <visual>
-            <origin xyz="-0.02 0 -0.03" rpy="-1.57 0 -1.57"/>
+            <origin xyz="-0.02 0 -0.03" rpy="${-PI/2} 0 ${-PI/2}"/>
             <geometry>
                 <mesh filename="package://aster_description/meshes/Greifer/files/Robotic_Arm_Palm.stl" scale="0.001 0.001 0.001"/>
@@ -199,5 +217,5 @@
     <link name="lh_rotate_top_link" >
         <visual>
-            <origin xyz="-0.004 0 -0.03" rpy="-1.57 0 -1.57"/>
+            <origin xyz="-0.004 0 -0.03" rpy="${-PI/2} 0 ${-PI/2}"/>
             <geometry>
                 <mesh filename="package://aster_description/meshes/Greifer/files/Robotic_Arm_Palm_Top.stl" scale="0.001 0.001 0.001"/>
@@ -208,5 +226,5 @@
     <link name="lh_gripper1_link" >
         <visual>
-            <origin xyz="-0.005 0.016 -0.008" rpy="-1.57 0 -1.57"/>
+            <origin xyz="-0.005 0.016 -0.008" rpy="${-PI/2} 0 ${-PI/2}"/>
             <geometry>
                 <mesh filename="package://aster_description/meshes/Greifer/files/Robotic_Arm_Finger.stl" scale="0.001 0.001 0.001"/>
@@ -217,9 +235,27 @@
     <link name="lh_gripper2_link" >
         <visual>
-            <origin xyz="0.007 -0.016 -0.008" rpy="-1.57 0 1.57"/>
+            <origin xyz="0.007 -0.016 -0.008" rpy="${-PI/2} 0 ${PI/2}"/>
             <geometry>
                 <mesh filename="package://aster_description/meshes/Greifer/files/Robotic_Arm_Finger.stl" scale="0.001 0.001 0.001"/>
             </geometry>
             <material name="white"/>
+        </visual>
+    </link>
+    <link name="lh_gripper1_pad_link" >
+        <visual>
+            <origin xyz="-0.004 -0.0015 -0.0017" rpy="0 ${PI/2} 0"/>
+            <geometry>
+                <mesh filename="package://aster_description/meshes/Greifer/files/Robotic_Arm_Finger_Pad.stl" scale="0.001 0.001 0.001"/>
+            </geometry>
+            <material name="blue"/>
+        </visual>
+    </link>
+    <link name="lh_gripper2_pad_link" >
+        <visual>
+            <origin xyz="0.005 0.0015 -0.0017" rpy="${PI} ${PI/2} 0"/>
+            <geometry>
+                <mesh filename="package://aster_description/meshes/Greifer/files/Robotic_Arm_Finger_Pad.stl" scale="0.001 0.001 0.001"/>
+            </geometry>
+            <material name="blue"/>
         </visual>
     </link>
@@ -263,5 +299,5 @@
         <child link="neck_link"/>
         <axis xyz="0 0 1 "/>
-        <limit lower="-1.57" upper="1.57" velocity="50.0" effort="1000.0"/>
+        <limit lower="${-PI/2}" upper="${PI/2}" velocity="50.0" effort="1000.0"/>
         <origin xyz="0 0 0.1" rpy="0 0 0"/>
     </joint>
@@ -278,5 +314,5 @@
         <child link="shoulder_rh_link"/>
         <axis xyz="0 1 0"/>
-        <limit lower="-1.57" upper="1.57" velocity="50.0" effort="1000.0"/>
+        <limit lower="${-PI/2}" upper="${PI/2}" velocity="50.0" effort="1000.0"/>
         <origin xyz="0.0 -0.085 0.05" rpy="0 0 0"/>
     </joint>
@@ -285,5 +321,5 @@
         <child link="sh_rh_lift_link"/>
         <axis xyz="1 0 0"/>
-        <limit lower="-1.57" upper="0" velocity="50.0" effort="1000.0"/>
+        <limit lower="${-PI/2}" upper="0" velocity="50.0" effort="1000.0"/>
         <origin xyz="-0.008 -0.027 0" rpy="0 0 0"/>
     </joint>
@@ -292,5 +328,5 @@
         <child link="sh_rh_rotate_link"/>
         <axis xyz="0 0 1"/>
-        <limit lower="-1.57" upper="1.57" velocity="50.0" effort="1000.0"/>
+        <limit lower="${-PI/2}" upper="${PI/2}" velocity="50.0" effort="1000.0"/>
         <origin xyz="0 0 -0.04" rpy="0 0 0"/>
     </joint>
@@ -299,5 +335,5 @@
         <child link="elbow_rh_link"/>
         <axis xyz="0 1 0"/>
-        <limit lower="-1.57" upper="0" velocity="50.0" effort="1000.0"/>
+        <limit lower="${-PI/2}" upper="0" velocity="50.0" effort="1000.0"/>
         <origin xyz="0 0 -0.13" rpy="0 0 0"/>
     </joint>
@@ -307,5 +343,5 @@
         <child link="rh_rotate_link"/>
         <axis xyz="0 0 1"/>
-        <limit lower="0" upper="1.57" velocity="50.0" effort="1000.0"/>
+        <limit lower="0" upper="${PI/2}" velocity="50.0" effort="1000.0"/>
         <origin xyz="0 -0.01 -0.13" rpy="0 0 0"/>
     </joint>
@@ -319,5 +355,5 @@
         <child link="rh_gripper1_link"/>
         <axis xyz="1 0 0"/>
-        <limit lower="-0.76" upper="0" velocity="50.0" effort="1000.0"/>
+        <limit lower="${-PI/6}" upper="0" velocity="50.0" effort="1000.0"/>
         <origin xyz="-0.015 -0.02 -0.048" rpy="0 0 0"/>
     </joint>
@@ -327,6 +363,16 @@
         <child link="rh_gripper2_link"/>
         <axis xyz="1 0 0"/>
-        <limit lower="0" upper="0.76" velocity="50.0" effort="1000.0"/>
+        <limit lower="0" upper="${PI/6}" velocity="50.0" effort="1000.0"/>
         <origin xyz="-0.015 0.02 -0.048" rpy="0 0 0"/>
+    </joint>
+    <joint name="virtual_8_joint" type="fixed">
+        <parent link="rh_gripper1_link"/>
+        <child link="rh_gripper1_pad_link"/>
+        <origin xyz="0 0.015 -0.041" rpy="0.0 0.0 0.0"/>
+    </joint>
+    <joint name="virtual_9_joint" type="fixed">
+        <parent link="rh_gripper2_link"/>
+        <child link="rh_gripper2_pad_link"/>
+        <origin xyz="0 -0.015 -0.041" rpy="0.0 0.0 0.0"/>
     </joint>
     <!-- Left Arm Joints-->
@@ -335,5 +381,5 @@
         <child link="shoulder_lh_link"/>
         <axis xyz="0 1 0"/>
-        <limit lower="-1.57" upper="1.57" velocity="50.0" effort="1000.0"/>
+        <limit lower="${-PI/2}" upper="${PI/2}" velocity="50.0" effort="1000.0"/>
         <origin xyz="0.0 0.085 0.05" rpy="0 0 0"/>
     </joint>
@@ -342,5 +388,5 @@
         <child link="sh_lh_lift_link"/>
         <axis xyz="1 0 0"/>
-        <limit lower="0" upper="1.57" velocity="50.0" effort="1000.0"/>
+        <limit lower="0" upper="${PI/2}" velocity="50.0" effort="1000.0"/>
         <origin xyz="-0.008 0.027 0" rpy="0 0 0"/>
     </joint>
@@ -349,5 +395,5 @@
         <child link="sh_lh_rotate_link"/>
         <axis xyz="0 0 1"/>
-        <limit lower="-1.57" upper="1.57" velocity="50.0" effort="1000.0"/>
+        <limit lower="${-PI/2}" upper="${PI/2}" velocity="50.0" effort="1000.0"/>
         <origin xyz="0 0 -0.04" rpy="0 0 0"/>
     </joint>
@@ -356,5 +402,5 @@
         <child link="elbow_lh_link"/>
         <axis xyz="0 1 0"/>
-        <limit lower="-1.57" upper="0" velocity="50.0" effort="1000.0"/>
+        <limit lower="${-PI/2}" upper="0" velocity="50.0" effort="1000.0"/>
         <origin xyz="0 0 -0.13" rpy="0 0 0"/>
     </joint>
@@ -364,5 +410,5 @@
         <child link="lh_rotate_link"/>
         <axis xyz="0 0 1"/>
-        <limit lower="-1.57" upper="0" velocity="50.0" effort="1000.0"/>
+        <limit lower="${-PI/2}" upper="0" velocity="50.0" effort="1000.0"/>
         <origin xyz="0 0.015 -0.13" rpy="0 0 0"/>
     </joint>
@@ -376,5 +422,5 @@
         <child link="lh_gripper1_link"/>
         <axis xyz="1 0 0"/>
-        <limit lower="-0.76" upper="0" velocity="50.0" effort="1000.0"/>
+        <limit lower="${-PI/6}" upper="0" velocity="50.0" effort="1000.0"/>
         <origin xyz="-0.015 -0.02 -0.048" rpy="0 0 0"/>
     </joint>
@@ -384,6 +430,16 @@
         <child link="lh_gripper2_link"/>
         <axis xyz="1 0 0"/>
-        <limit lower="0" upper="0.76" velocity="50.0" effort="1000.0"/>
+        <limit lower="0" upper="${PI/6}" velocity="50.0" effort="1000.0"/>
         <origin xyz="-0.015 0.02 -0.048" rpy="0 0 0"/>
+    </joint>
+    <joint name="virtual_11_joint" type="fixed">
+        <parent link="lh_gripper1_link"/>
+        <child link="lh_gripper1_pad_link"/>
+        <origin xyz="0 0.015 -0.041" rpy="0.0 0.0 0.0"/>
+    </joint>
+    <joint name="virtual_12_joint" type="fixed">
+        <parent link="lh_gripper2_link"/>
+        <child link="lh_gripper2_pad_link"/>
+        <origin xyz="0 -0.015 -0.041" rpy="0.0 0.0 0.0"/>
     </joint>
     <!-- Right Leg Joints-->

Commit message: nur noch die füsse

File: aster_description/urdf/aster.xacro (robot description, xacro)
@@ -261,5 +261,41 @@
     </link>
     <!-- Right Leg-->
+    <link name="hip_rh_link">
+        <visual>
+            <origin xyz="0.0023 -0.015 -0.1748" rpy="0 0 0"/>
+            <geometry>
+                <mesh filename="package://aster_description/meshes/Right_Leg_Upper.stl" scale="0.001 0.001 0.001"/>
+            </geometry>
+            <material name="white"/>
+        </visual>
+    </link>
+    <link name="knie_rh_link" >
+        <visual>
+            <origin xyz="0.0025 0 -0.1765" rpy="0 0 0"/>
+            <geometry>
+                <mesh filename="package://aster_description/meshes/Right_Leg_Lower.stl" scale="0.001 0.001 0.001"/>
+            </geometry>
+            <material name="white"/>
+        </visual>
+    </link>
     <!-- Left Leg-->
+    <link name="hip_lh_link">
+        <visual>
+            <origin xyz="0.0023 0.015 -0.1748" rpy="0 0 0"/>
+            <geometry>
+                <mesh filename="package://aster_description/meshes/Left_Leg_Upper.stl" scale="0.001 0.001 0.001"/>
+            </geometry>
+            <material name="white"/>
+        </visual>
+    </link>
+    <link name="knie_lh_link" >
+        <visual>
+            <origin xyz="0.0025 0 -0.1765" rpy="0 0 0"/>
+            <geometry>
+                <mesh filename="package://aster_description/meshes/Left_Lower_Leg.stl" scale="0.001 0.001 0.001"/>
+            </geometry>
+            <material name="white"/>
+        </visual>
+    </link>
                     <!-- ######  JOINTS  ######-->
     <!-- Base Virtual Joints-->
@@ -444,4 +480,32 @@
     </joint>
     <!-- Right Leg Joints-->
+    <joint name="joint_15" type="revolute">
+        <parent link="hip_link"/>
+        <child link="hip_rh_link"/>
+        <axis xyz="0 1 0"/>
+        <limit lower="${-PI/2}" upper="${PI/2}" velocity="50.0" effort="1000.0"/>
+        <origin xyz="-0.007 -0.042 -0.024" rpy="0 0 0"/>
+    </joint>
+    <joint name="joint_16" type="revolute">
+        <parent link="hip_rh_link"/>
+        <child link="knie_rh_link"/>
+        <axis xyz="0 1 0"/>
+        <limit lower="0" upper="${PI/2}" velocity="50.0" effort="1000.0"/>
+        <origin xyz="0 0 -0.185" rpy="0 0 0"/>
+    </joint>
     <!-- Left Leg Joints-->
+    <joint name="joint_18" type="revolute">
+        <parent link="hip_link"/>
+        <child link="hip_lh_link"/>
+        <axis xyz="0 1 0"/>
+        <limit lower="${-PI/2}" upper="${PI/2}" velocity="50.0" effort="1000.0"/>
+        <origin xyz="-0.007 0.042 -0.024" rpy="0 0 0"/>
+    </joint>
+    <joint name="joint_19" type="revolute">
+        <parent link="hip_lh_link"/>
+        <child link="knie_lh_link"/>
+        <axis xyz="0 1 0"/>
+        <limit lower="0" upper="${PI/2}" velocity="50.0" effort="1000.0"/>
+        <origin xyz="0 0 -0.185" rpy="0 0 0"/>
+    </joint>
 </robot>

Commit message: raw urdf is ready. now collission and iniertial

File: aster_description/urdf/aster.xacro (robot description, xacro)
@@ -279,4 +279,13 @@
         </visual>
     </link>
+    <link name="foot_rh_link" >
+        <visual>
+            <origin xyz="0.03 -0.0025 -0.035" rpy="0 0 0"/>
+            <geometry>
+                <mesh filename="package://aster_description/meshes/Right_Leg_Foot.stl" scale="0.001 0.001 0.001"/>
+            </geometry>
+            <material name="blue"/>
+        </visual>
+    </link>
     <!-- Left Leg-->
     <link name="hip_lh_link">
@@ -296,4 +305,13 @@
             </geometry>
             <material name="white"/>
+        </visual>
+    </link>
+    <link name="foot_lh_link" >
+        <visual>
+            <origin xyz="0.03 0.0025 -0.035" rpy="0 0 0"/>
+            <geometry>
+                <mesh filename="package://aster_description/meshes/Left_Leg_Foot.stl" scale="0.001 0.001 0.001"/>
+            </geometry>
+            <material name="blue"/>
         </visual>
     </link>
@@ -308,5 +326,5 @@
         <parent link="base_link"/>
         <child link="base_holder_link"/>
-        <origin xyz="0.0 0.0 0.65" rpy="0.0 0.0 0.0"/>
+        <origin xyz="0.0 0.0 0.62" rpy="0.0 0.0 0.0"/>
     </joint>
     <joint name="virtual_3_joint" type="fixed">
@@ -494,4 +512,11 @@
         <origin xyz="0 0 -0.185" rpy="0 0 0"/>
     </joint>
+    <joint name="joint_17" type="revolute">
+        <parent link="knie_rh_link"/>
+        <child link="foot_rh_link"/>
+        <axis xyz="0 1 0"/>
+        <limit lower="${-PI/4}" upper="${PI/4}" velocity="50.0" effort="1000.0"/>
+        <origin xyz="0 0 -0.18" rpy="0 0 0"/>
+    </joint>
     <!-- Left Leg Joints-->
     <joint name="joint_18" type="revolute">
@@ -509,3 +534,10 @@
         <origin xyz="0 0 -0.185" rpy="0 0 0"/>
     </joint>
+    <joint name="joint_20" type="revolute">
+        <parent link="knie_lh_link"/>
+        <child link="foot_lh_link"/>
+        <axis xyz="0 1 0"/>
+        <limit lower="${-PI/4}" upper="${PI/4}" velocity="50.0" effort="1000.0"/>
+        <origin xyz="0 0 -0.18" rpy="0 0 0"/>
+    </joint>
 </robot>

Commit message: added face and colors like in real

File: aster_description/urdf/aster.xacro (robot description, xacro)
@@ -1,4 +1,5 @@
 <?xml version="1.0"?>
 <robot xmlns:xacro="http://www.ros.org/wiki/xacro" >
+    <!-- <xacro:default_inertial mass="0.3"/> -->
     <link name="world"/>
     <link name="base_link">
@@ -36,5 +37,5 @@
                 <mesh filename="package://aster_description/meshes/Chest.stl" scale="0.001 0.001 0.001"/>
             </geometry>
-            <material name="blue"/>
+            <material name="black"/>
         </visual>
     </link>
@@ -45,5 +46,5 @@
                 <mesh filename="package://aster_description/meshes/Spine.stl" scale="0.001 0.001 0.001"/>
             </geometry>
-            <material name="blue"/>
+            <material name="white"/>
         </visual>
     </link>
@@ -54,5 +55,5 @@
                 <mesh filename="package://aster_description/meshes/Hips.stl" scale="0.001 0.001 0.001"/>
             </geometry>
-            <material name="blue"/>
+            <material name="white"/>
         </visual>
     </link>
@@ -76,4 +77,13 @@
         </visual>
     </link>
+    <link name="face_link">
+        <visual>
+            <origin xyz="0.038 0 -0.0125" rpy="1.57 0 1.57"/>
+            <geometry>
+                <mesh filename="package://aster_description/meshes/ownStls/Face_OLED_PiCam.stl" scale="0.001 0.001 0.001"/>
+            </geometry>
+            <material name="black"/>
+        </visual>
+    </link>
     <!-- Right Arm-->
     <link name="shoulder_rh_link">
@@ -156,5 +166,5 @@
                 <mesh filename="package://aster_description/meshes/Greifer/files/Robotic_Arm_Finger_Pad.stl" scale="0.001 0.001 0.001"/>
             </geometry>
-            <material name="blue"/>
+            <material name="black"/>
         </visual>
     </link>
@@ -165,5 +175,5 @@
                 <mesh filename="package://aster_description/meshes/Greifer/files/Robotic_Arm_Finger_Pad.stl" scale="0.001 0.001 0.001"/>
             </geometry>
-            <material name="blue"/>
+            <material name="black"/>
         </visual>
     </link>
@@ -248,5 +258,5 @@
                 <mesh filename="package://aster_description/meshes/Greifer/files/Robotic_Arm_Finger_Pad.stl" scale="0.001 0.001 0.001"/>
             </geometry>
-            <material name="blue"/>
+            <material name="black"/>
         </visual>
     </link>
@@ -257,5 +267,5 @@
                 <mesh filename="package://aster_description/meshes/Greifer/files/Robotic_Arm_Finger_Pad.stl" scale="0.001 0.001 0.001"/>
             </geometry>
-            <material name="blue"/>
+            <material name="black"/>
         </visual>
     </link>
@@ -285,5 +295,5 @@
                 <mesh filename="package://aster_description/meshes/Right_Leg_Foot.stl" scale="0.001 0.001 0.001"/>
             </geometry>
-            <material name="blue"/>
+            <material name="black"/>
         </visual>
     </link>
@@ -304,5 +314,5 @@
                 <mesh filename="package://aster_description/meshes/Left_Lower_Leg.stl" scale="0.001 0.001 0.001"/>
             </geometry>
-            <material name="white"/>
+            <material name="black"/>
         </visual>
     </link>
@@ -313,5 +323,5 @@
                 <mesh filename="package://aster_description/meshes/Left_Leg_Foot.stl" scale="0.001 0.001 0.001"/>
             </geometry>
-            <material name="blue"/>
+            <material name="black"/>
         </visual>
     </link>
@@ -362,4 +372,9 @@
         <limit lower="-0.5" upper="0.3" velocity="50.0" effort="1000.0"/>
         <origin xyz="0 0 0.01" rpy="0 0 0"/>
+    </joint>
+    <joint name="face_joint" type="fixed">
+        <parent link="head_link"/>
+        <child link="face_link"/>
+        <origin xyz="0.0 0.0 0.0375" rpy="0.0 0.0 0.0"/>
     </joint>
     <!-- Right Arm Joints-->

File: aster_description/urdf/material.xacro (robot description, xacro)
@@ -10,4 +10,7 @@
         <color rgba="0.0 0.0 1.0 0.8"/>
     </material>
+    <material name="black">
+        <color rgba="0.0 0.0 0.0 1"/>
+    </material>
     <!-- Inertial für Stl körper-->
     <xacro:macro name="default_inertial" params="mass"> <!-- <xacro:default_inertial mass="1.0"/> -->
