Commit message: fehler suche gazebo läd nicht richtig

File: aster_description/urdf/aster.xacro (robot description, xacro)
@@ -682,5 +682,5 @@
         <origin xyz="-0.015 -0.02 -0.048" rpy="0 0 0"/>
     </joint>
-    <joint name="joint_8_m" type="revolute">
+    <joint name="joint_21" type="revolute">
         <mimic joint="joint_8" multiplier="-1"/>
         <parent link="rh_rotate_link"/>
@@ -749,5 +749,5 @@
         <origin xyz="-0.015 -0.02 -0.048" rpy="0 0 0"/>
     </joint>
-    <joint name="joint_14_m" type="revolute">
+    <joint name="joint_22" type="revolute">
         <mimic joint="joint_14" multiplier="-1"/>
         <parent link="lh_rotate_link"/>

File: aster_description/urdf/aster_ros2_control.xacro (robot description, xacro)
@@ -8,5 +8,5 @@
         <!-- ros2_control Gazebo
         <xacro:if value="$(arg is_sim)">
-            <joint name="joint_8_m">
+            <joint name="joint_21">
                 <param name="mimic">joint_8</param>
                 <param name="multiplier">-1</param>
@@ -16,5 +16,5 @@
                 </command_interface>
             </joint>
-            <joint name="joint_14_m">
+            <joint name="joint_22">
                 <param name="mimic">joint_14</param>
                 <param name="multiplier">-1</param>
@@ -87,5 +87,5 @@
             <state_interface name="position" />
         </joint>
-        <joint name="joint_8_m">
+        <joint name="joint_21">
             <param name="mimic">joint_8</param>
             <param name="multiplier">-1</param>
@@ -137,5 +137,5 @@
             <state_interface name="position" />
         </joint>
-        <joint name="joint_14_m">
+        <joint name="joint_22">
             <param name="mimic">joint_14</param>
             <param name="multiplier">-1</param>

File: aster_description/urdf/material.xacro (robot description, xacro)
@@ -1,15 +1,15 @@
 <?xml version="1.0"?>
-<robot xmlns:xacro="http://www.ros.org/wiki/xacro" >
+<robot xmlns:xacro="http://www.ros.org/wiki/xacro">
     <xacro:property name="PI" value="3.14159265359" />
     <xacro:property name="effort" value="30.0" />
     <xacro:property name="velocity" value="10.0" />
     <material name="white">
-        <color rgba="1 1 1 0.8"/>
+        <color rgba="1 1 1 0.8" />
     </material>
     <material name="blue">
-        <color rgba="0.0 0.0 1.0 0.8"/>
+        <color rgba="0.0 0.0 1.0 0.8" />
     </material>
     <material name="black">
-        <color rgba="0.0 0.0 0.0 1"/>
+        <color rgba="0.0 0.0 0.0 1" />
     </material>
     <!-- Inertial für Stl körper-->
@@ -18,6 +18,6 @@
             <mass value="${mass}" />
             <inertia ixx="0.0001" ixy="0.0" ixz="0.0"
-                     iyy="0.0001" iyz="0.0"
-                     izz="0.0001" />
+                iyy="0.0001" iyz="0.0"
+                izz="0.0001" />
         </inertial>
     </xacro:macro>
@@ -26,6 +26,6 @@
             <mass value="${mass}" />
             <inertia ixx="0.00001" ixy="0.0" ixz="0.0"
-                     iyy="0.00001" iyz="0.0"
-                     izz="0.00001" />
+                iyy="0.00001" iyz="0.0"
+                izz="0.00001" />
         </inertial>
     </xacro:macro>

Commit message: searching fail

File: aster_description/urdf/aster.xacro (robot description, xacro)
@@ -1,4 +1,34 @@
 <?xml version="1.0"?>
-<robot xmlns:xacro="http://www.ros.org/wiki/xacro" >
+<robot xmlns:xacro="http://www.ros.org/wiki/xacro" name="aster">
+    <xacro:property name="PI" value="3.14159265359" />
+    <xacro:property name="effort" value="30.0" />
+    <xacro:property name="velocity" value="10.0" />
+    <material name="white">
+        <color rgba="1.0 1.0 1.0 0.8" />
+    </material>
+    <material name="blue">
+        <color rgba="0.0 0.0 1.0 0.8" />
+    </material>
+    <material name="black">
+        <color rgba="0.0 0.0 0.0 1.0" />
+    </material>
+    <!-- Inertial für Stl körper-->
+    <xacro:macro name="default_inertial" params="mass"> <!-- <xacro:default_inertial mass="1.0"/> -->
+        <inertial>
+            <mass value="${mass}" />
+            <inertia ixx="0.0001" ixy="0.0" ixz="0.0"
+                iyy="0.0001" iyz="0.0"
+                izz="0.0001" />
+        </inertial>
+    </xacro:macro>
+    <xacro:macro name="default_inertial_1" params="masse"> <!-- <xacro:default_inertial_1
+        mass="1.0"/> -->
+        <inertial>
+            <mass value="${masse}" />
+            <inertia ixx="0.00001" ixy="0.0" ixz="0.0"
+                iyy="0.00001" iyz="0.0"
+                izz="0.00001" />
+        </inertial>
+    </xacro:macro>
     <!-- <xacro:default_inertial mass="0.3"/> -->
     <!-- <xacro:default_inertial_1 mass="0.03"/> -->
@@ -6,5 +36,5 @@
         <transmission name="transmission_${number}">
             <plugin>transmission_interface/SimpleTransmission</plugin>
-            <actuator name="motor_${number}" role="actuator1"/>
+            <actuator name="motor_${number}" role="actuator1" />
             <joint name="joint_${number}" role="joint1">
                 <mechanical_reduction>1.0</mechanical_reduction>
@@ -12,231 +42,261 @@
         </transmission>
     </xacro:macro>
-    <link name="world"/>
+    <link name="world" />
     <link name="base_link">
         <visual>
-            <origin xyz="0.0 0.0 0.0" rpy="0.0 0.0 0.0"/>
-            <geometry>
-                <mesh filename="package://aster_description/meshes/ownStls/standBase.stl" scale="0.001 0.001 0.001"/>
-            </geometry>
-            <material name="white"/>
-        </visual>
-        <collision>
-            <origin xyz="0.0 0.0 0.0" rpy="0.0 0.0 0.0"/>
-            <geometry>
-                <mesh filename="package://aster_description/meshes/ownStls/standBase.stl" scale="0.001 0.001 0.001"/>
-            </geometry>
-        </collision>
-        <xacro:default_inertial mass="3.3"/>
+            <origin xyz="0.0 0.0 0.0" rpy="0.0 0.0 0.0" />
+            <geometry>
+                <mesh filename="package://aster_description/meshes/ownStls/standBase.stl"
+                    scale="0.001 0.001 0.001" />
+            </geometry>
+            <material name="white" />
+        </visual>
+        <collision>
+            <origin xyz="0.0 0.0 0.0" rpy="0.0 0.0 0.0" />
+            <geometry>
+                <mesh filename="package://aster_description/meshes/ownStls/standBase.stl"
+                    scale="0.001 0.001 0.001" />
+            </geometry>
+        </collision>
+        <xacro:default_inertial mass="3.3" />
     </link>
     <!-- Base-->
     <link name="base_holder_link">
         <visual>
-            <origin xyz="0.0 0.0 -0.02" rpy="0.0 0.0 ${-PI/2}"/>
-            <geometry>
-                <mesh filename="package://aster_description/meshes/subStuff/RohrHalter_v2.stl" scale="0.001 0.001 0.001"/>
-            </geometry>
-            <material name="white"/>
-        </visual>
-        <collision>
-            <origin xyz="0.0 0.0 -0.02" rpy="0.0 0.0 ${-PI/2}"/>
-            <geometry>
-                <mesh filename="package://aster_description/meshes/subStuff/RohrHalter_v2.stl" scale="0.001 0.001 0.001"/>
-            </geometry>
-        </collision>
-        <xacro:default_inertial mass="0.3"/>
+            <origin xyz="0.0 0.0 -0.02" rpy="0.0 0.0 ${-PI/2}" />
+            <geometry>
+                <mesh filename="package://aster_description/meshes/subStuff/RohrHalter_v2.stl"
+                    scale="0.001 0.001 0.001" />
+            </geometry>
+            <material name="white" />
+        </visual>
+        <collision>
+            <origin xyz="0.0 0.0 -0.02" rpy="0.0 0.0 ${-PI/2}" />
+            <geometry>
+                <mesh filename="package://aster_description/meshes/subStuff/RohrHalter_v2.stl"
+                    scale="0.001 0.001 0.001" />
+            </geometry>
+        </collision>
+        <xacro:default_inertial mass="0.3" />
     </link>
     <link name="chest_bone_link">
         <visual>
-            <origin xyz="0.0 0.0 0.0" rpy="0.0 0.0 0.0"/>
-            <geometry>
-                <mesh filename="package://aster_description/meshes/Spine_Connector.stl" scale="0.001 0.001 0.001"/>
-            </geometry>
-            <material name="white"/>
-        </visual>
-        <collision>
-            <origin xyz="0.0 0.0 0.0" rpy="0.0 0.0 0.0"/>
-            <geometry>
-                <mesh filename="package://aster_description/meshes/Spine_Connector.stl" scale="0.001 0.001 0.001"/>
-            </geometry>
-        </collision>
-        <xacro:default_inertial mass="0.3"/>
+            <origin xyz="0.0 0.0 0.0" rpy="0.0 0.0 0.0" />
+            <geometry>
+                <mesh filename="package://aster_description/meshes/Spine_Connector.stl"
+                    scale="0.001 0.001 0.001" />
+            </geometry>
+            <material name="white" />
+        </visual>
+        <collision>
+            <origin xyz="0.0 0.0 0.0" rpy="0.0 0.0 0.0" />
+            <geometry>
+                <mesh filename="package://aster_description/meshes/Spine_Connector.stl"
+                    scale="0.001 0.001 0.001" />
+            </geometry>
+        </collision>
+        <xacro:default_inertial mass="0.3" />
     </link>
     <link name="chest_link">
         <visual>
-            <origin xyz="0.0 0.0 -0.012" rpy="0.0 0.0 0.0"/>
-            <geometry>
-                <mesh filename="package://aster_description/meshes/Chest.stl" scale="0.001 0.001 0.001"/>
-            </geometry>
-            <material name="black"/>
-        </visual>
-        <collision>
-            <origin xyz="0.0 0.0 -0.012" rpy="0.0 0.0 0.0"/>
-            <geometry>
-                <mesh filename="package://aster_description/meshes/Chest.stl" scale="0.001 0.001 0.001"/>
-            </geometry>
-        </collision>
-        <xacro:default_inertial mass="0.3"/>
+            <origin xyz="0.0 0.0 -0.012" rpy="0.0 0.0 0.0" />
+            <geometry>
+                <mesh filename="package://aster_description/meshes/Chest.stl"
+                    scale="0.001 0.001 0.001" />
+            </geometry>
+            <material name="black" />
+        </visual>
+        <collision>
+            <origin xyz="0.0 0.0 -0.012" rpy="0.0 0.0 0.0" />
+            <geometry>
+                <mesh filename="package://aster_description/meshes/Chest.stl"
+                    scale="0.001 0.001 0.001" />
+            </geometry>
+        </collision>
+        <xacro:default_inertial mass="0.3" />
     </link>
     <link name="backbone_link">
         <visual>
-            <origin xyz="-0.003 0.0 -0.085" rpy="0.0 0.0 0.0"/>
-            <geometry>
-                <mesh filename="package://aster_description/meshes/Spine.stl" scale="0.001 0.001 0.001"/>
-            </geometry>
-            <material name="white"/>
-        </visual>
-        <collision>
-            <origin xyz="-0.003 0.0 -0.085" rpy="0.0 0.0 0.0"/>
-            <geometry>
-                <mesh filename="package://aster_description/meshes/Spine.stl" scale="0.001 0.001 0.001"/>
-            </geometry>
-        </collision>
-        <xacro:default_inertial mass="0.3"/>
+            <origin xyz="-0.003 0.0 -0.085" rpy="0.0 0.0 0.0" />
+            <geometry>
+                <mesh filename="package://aster_description/meshes/Spine.stl"
+                    scale="0.001 0.001 0.001" />
+            </geometry>
+            <material name="white" />
+        </visual>
+        <collision>
+            <origin xyz="-0.003 0.0 -0.085" rpy="0.0 0.0 0.0" />
+            <geometry>
+                <mesh filename="package://aster_description/meshes/Spine.stl"
+                    scale="0.001 0.001 0.001" />
+            </geometry>
+        </collision>
+        <xacro:default_inertial mass="0.3" />
     </link>
     <link name="hip_link">
         <visual>
-            <origin xyz="-0.005 0.0 0.003" rpy="0.0 0.0 0.0"/>
-            <geometry>
-                <mesh filename="package://aster_description/meshes/Hips.stl" scale="0.001 0.001 0.001"/>
-            </geometry>
-            <material name="white"/>
-        </visual>
-        <collision>
-            <origin xyz="-0.005 0.0 0.003" rpy="0.0 0.0 0.0"/>
-            <geometry>
-                <mesh filename="package://aster_description/meshes/Hips.stl" scale="0.001 0.001 0.001"/>
-            </geometry>
-        </collision>
-        <xacro:default_inertial mass="0.3"/>
-    </link>
-   <!-- Head-->
+            <origin xyz="-0.005 0.0 0.003" rpy="0.0 0.0 0.0" />
+            <geometry>
+                <mesh filename="package://aster_description/meshes/Hips.stl"
+                    scale="0.001 0.001 0.001" />
+            </geometry>
+            <material name="white" />
+        </visual>
+        <collision>
+            <origin xyz="-0.005 0.0 0.003" rpy="0.0 0.0 0.0" />
+            <geometry>
+                <mesh filename="package://aster_description/meshes/Hips.stl"
+                    scale="0.001 0.001 0.001" />
+            </geometry>
+        </collision>
+        <xacro:default_inertial mass="0.3" />
+    </link>
+    <!-- Head-->
     <link name="neck_link">
         <visual>
-            <origin xyz="0.0 0.0 -0.012" rpy="0.0 0.0 0.0"/>
-            <geometry>
-                <mesh filename="package://aster_description/meshes/Head_Neck.stl" scale="0.001 0.001 0.001"/>
-            </geometry>
-            <material name="blue"/>
-        </visual>
-        <collision>
-            <origin xyz="0.0 0.0 -0.012" rpy="0.0 0.0 0.0"/>
-            <geometry>
-                <mesh filename="package://aster_description/meshes/Head_Neck.stl" scale="0.001 0.001 0.001"/>
-            </geometry>
-        </collision>
-        <xacro:default_inertial mass="0.3"/>
+            <origin xyz="0.0 0.0 -0.012" rpy="0.0 0.0 0.0" />
+            <geometry>
+                <mesh filename="package://aster_description/meshes/Head_Neck.stl"
+                    scale="0.001 0.001 0.001" />
+            </geometry>
+            <material name="blue" />
+        </visual>
+        <collision>
+            <origin xyz="0.0 0.0 -0.012" rpy="0.0 0.0 0.0" />
+            <geometry>
+                <mesh filename="package://aster_description/meshes/Head_Neck.stl"
+                    scale="0.001 0.001 0.001" />
+            </geometry>
+        </collision>
+        <xacro:default_inertial mass="0.3" />
     </link>
     <link name="head_link">
         <visual>
-            <origin xyz="0.0 0.0 -0.012" rpy="0.0 0.0 0.0"/>
-            <geometry>
-                <mesh filename="package://aster_description/meshes/Head_Back.stl" scale="0.001 0.001 0.001"/>
-            </geometry>
-            <material name="white"/>
-        </visual>
-        <collision>
-            <origin xyz="0.0 0.0 -0.012" rpy="0.0 0.0 0.0"/>
-            <geometry>
-                <mesh filename="package://aster_description/meshes/Head_Back.stl" scale="0.001 0.001 0.001"/>
-            </geometry>
-        </collision>
-        <xacro:default_inertial mass="0.3"/>
+            <origin xyz="0.0 0.0 -0.012" rpy="0.0 0.0 0.0" />
+            <geometry>
+                <mesh filename="package://aster_description/meshes/Head_Back.stl"
+                    scale="0.001 0.001 0.001" />
+            </geometry>
+            <material name="white" />
+        </visual>
+        <collision>
+            <origin xyz="0.0 0.0 -0.012" rpy="0.0 0.0 0.0" />
+            <geometry>
+                <mesh filename="package://aster_description/meshes/Head_Back.stl"
+                    scale="0.001 0.001 0.001" />
+            </geometry>
+        </collision>
+        <xacro:default_inertial mass="0.3" />
     </link>
     <link name="face_link">
         <visual>
-            <origin xyz="0.038 0 -0.0125" rpy="1.57 0 1.57"/>
-            <geometry>
-                <mesh filename="package://aster_description/meshes/ownStls/Face_OLED_PiCam.stl" scale="0.001 0.001 0.001"/>
-            </geometry>
-            <material name="black"/>
-        </visual>
-        <collision>
-            <origin xyz="0.038 0 -0.0125" rpy="1.57 0 1.57"/>
-            <geometry>
-                <mesh filename="package://aster_description/meshes/ownStls/Face_OLED_PiCam.stl" scale="0.001 0.001 0.001"/>
-            </geometry>
-        </collision>
-        <xacro:default_inertial mass="0.3"/>
+            <origin xyz="0.038 0 -0.0125" rpy="1.57 0 1.57" />
+            <geometry>
+                <mesh filename="package://aster_description/meshes/ownStls/Face_OLED_PiCam.stl"
+                    scale="0.001 0.001 0.001" />
+            </geometry>
+            <material name="black" />
+        </visual>
+        <collision>
+            <origin xyz="0.038 0 -0.0125" rpy="1.57 0 1.57" />
+            <geometry>
+                <mesh filename="package://aster_description/meshes/ownStls/Face_OLED_PiCam.stl"
+                    scale="0.001 0.001 0.001" />
+            </geometry>
+        </collision>
+        <xacro:default_inertial mass="0.3" />
     </link>
     <!-- Right Arm-->
     <link name="shoulder_rh_link">
         <visual>
-            <origin xyz="-0.01 -0.018 -0.023" rpy="0.0 0.0 0.0"/>
-            <geometry>
-                <mesh filename="package://aster_description/meshes/Rigth_Arm_Shoulder_Connector.stl" scale="0.001 0.001 0.001"/>
-            </geometry>
-            <material name="white"/>
-        </visual>
-        <collision>
-            <origin xyz="-0.01 -0.018 -0.023" rpy="0.0 0.0 0.0"/>
-            <geometry>
-                <mesh filename="package://aster_description/meshes/Rigth_Arm_Shoulder_Connector.stl" scale="0.001 0.001 0.001"/>
-            </geometry>
-        </collision>
-        <xacro:default_inertial mass="0.3"/>
+            <origin xyz="-0.01 -0.018 -0.023" rpy="0.0 0.0 0.0" />
+            <geometry>
+                <mesh filename="package://aster_description/meshes/Rigth_Arm_Shoulder_Connector.stl"
+                    scale="0.001 0.001 0.001" />
+            </geometry>
+            <material name="white" />
+        </visual>
+        <collision>
+            <origin xyz="-0.01 -0.018 -0.023" rpy="0.0 0.0 0.0" />
+            <geometry>
+                <mesh filename="package://aster_description/meshes/Rigth_Arm_Shoulder_Connector.stl"
+                    scale="0.001 0.001 0.001" />
+            </geometry>
+        </collision>
+        <xacro:default_inertial mass="0.3" />
     </link>
     <link name="sh_rh_lift_link">
         <visual>
-            <origin xyz="0 0.108 -0.6625" rpy="0.0 0.0 0.0"/>
-            <geometry>
-                <mesh filename="package://aster_description/meshes/Right_Arm_Shoulder.stl" scale="0.001 0.001 0.001"/>
-            </geometry>
-            <material name="white"/>
-        </visual>
-        <collision>
-            <origin xyz="0 0.108 -0.6625" rpy="0.0 0.0 0.0"/>
-            <geometry>
-                <mesh filename="package://aster_description/meshes/Right_Arm_Shoulder.stl" scale="0.001 0.001 0.001"/>
-            </geometry>
-        </collision>
-        <xacro:default_inertial mass="0.3"/>
+            <origin xyz="0 0.108 -0.6625" rpy="0.0 0.0 0.0" />
+            <geometry>
+                <mesh filename="package://aster_description/meshes/Right_Arm_Shoulder.stl"
+                    scale="0.001 0.001 0.001" />
+            </geometry>
+            <material name="white" />
+        </visual>
+        <collision>
+            <origin xyz="0 0.108 -0.6625" rpy="0.0 0.0 0.0" />
+            <geometry>
+                <mesh filename="package://aster_description/meshes/Right_Arm_Shoulder.stl"
+                    scale="0.001 0.001 0.001" />
+            </geometry>
+        </collision>
+        <xacro:default_inertial mass="0.3" />
     </link>
     <link name="sh_rh_rotate_link">
         <visual>
-            <origin xyz="0 0.108 0.51" rpy="${PI} 0 ${PI}"/>
-            <geometry>
-                <mesh filename="package://aster_description/meshes/Right_Arm_Upper.stl" scale="0.001 0.001 0.001"/>
-            </geometry>
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
File: aster_description/urdf/gazebo.xacro (robot description, xacro)
@@ -6,7 +6,6 @@
         <robot_param>robot_description</robot_param>
         <robot_param_node>robot_state_publisher</robot_param_node>
-        <parameters></parameters>
+        <parameters>$(find aster_controller)/config/controllers.yaml</parameters>
       </plugin>
     </gazebo>
-<!-- $(find aster_controller)/config/aster_controllers.yaml -->
 </robot>

File: aster_description/urdf/material.xacro (robot description, xacro)
@@ -1,9 +1,9 @@
 <?xml version="1.0"?>
-<robot xmlns:xacro="http://www.ros.org/wiki/xacro">
+<robot xmlns:xacro="http://www.ros.org/wiki/xacro" name="aster">
     <xacro:property name="PI" value="3.14159265359" />
     <xacro:property name="effort" value="30.0" />
     <xacro:property name="velocity" value="10.0" />
     <material name="white">
-        <color rgba="1 1 1 0.8" />
+        <color rgba="1.0 1.0 1.0 0.8" />
     </material>
     <material name="blue">
@@ -11,5 +11,5 @@
     </material>
     <material name="black">
-        <color rgba="0.0 0.0 0.0 1" />
+        <color rgba="0.0 0.0 0.0 1.0" />
     </material>
     <!-- Inertial für Stl körper-->
@@ -22,7 +22,7 @@
         </inertial>
     </xacro:macro>
-    <xacro:macro name="default_inertial_1" params="mass"> <!-- <xacro:default_inertial_1 mass="1.0"/> -->
+    <xacro:macro name="default_inertial_1" params="masse"> <!-- <xacro:default_inertial_1 mass="1.0"/> -->
         <inertial>
-            <mass value="${mass}" />
+            <mass value="${masse}" />
             <inertia ixx="0.00001" ixy="0.0" ixz="0.0"
                 iyy="0.00001" iyz="0.0"

File: aster_description/urdf/ros2_control.xacro (robot description, xacro)
@@ -23,5 +23,4 @@
             <hardware>
                 <plugin>aster_controller/asterInterface</plugin>
-                <param name="port">/dev/ttyUSB0</param>
             </hardware>
         </xacro:unless> -->
@@ -52,5 +51,5 @@
             <command_interface name="position">
                 <param name="min">-${PI / 2}</param>
-                <param name="max">0</param>
+                <param name="max">0.0</param>
             </command_interface>
             <state_interface name="position" />
@@ -66,5 +65,5 @@
             <command_interface name="position">
                 <param name="min">-${PI / 2}</param>
-                <param name="max">0</param>
+                <param name="max">0.0</param>
             </command_interface>
             <state_interface name="position" />
@@ -72,5 +71,5 @@
         <joint name="joint_7">
             <command_interface name="position">
-                <param name="min">0</param>
+                <param name="min">0.0</param>
                 <param name="max">${PI / 2}</param>
             </command_interface>
