Commit message: no clue. seaching

File: aster_description/urdf/aster.xacro (robot description, xacro)
@@ -1,34 +1,4 @@
 <?xml version="1.0"?>
 <robot xmlns:xacro="http://www.ros.org/wiki/xacro" name="aster">
-    <xacro:property name="PI" value="3.14159265359" />
-    <xacro:property name="effort" value="30.0" />
-    <xacro:property name="velocity" value="10.0" />
-    <material name="white">
-        <color rgba="1.0 1.0 1.0 0.8" />
-    </material>
-    <material name="blue">
-        <color rgba="0.0 0.0 1.0 0.8" />
-    </material>
-    <material name="black">
-        <color rgba="0.0 0.0 0.0 1.0" />
-    </material>
-    <!-- Inertial für Stl körper-->
-    <xacro:macro name="default_inertial" params="mass"> <!-- <xacro:default_inertial mass="1.0"/> -->
-        <inertial>
-            <mass value="${mass}" />
-            <inertia ixx="0.0001" ixy="0.0" ixz="0.0"
-                iyy="0.0001" iyz="0.0"
-                izz="0.0001" />
-        </inertial>
-    </xacro:macro>
-    <xacro:macro name="default_inertial_1" params="masse"> <!-- <xacro:default_inertial_1
-        mass="1.0"/> -->
-        <inertial>
-            <mass value="${masse}" />
-            <inertia ixx="0.00001" ixy="0.0" ixz="0.0"
-                iyy="0.00001" iyz="0.0"
-                izz="0.00001" />
-        </inertial>
-    </xacro:macro>
     <!-- <xacro:default_inertial mass="0.3"/> -->
     <!-- <xacro:default_inertial_1 mass="0.03"/> -->
@@ -191,5 +161,5 @@
     <link name="face_link">
         <visual>
-            <origin xyz="0.038 0 -0.0125" rpy="1.57 0 1.57" />
+            <origin xyz="0.038 0.0 -0.0125" rpy="1.57 0.0 1.57" />
             <geometry>
                 <mesh filename="package://aster_description/meshes/ownStls/Face_OLED_PiCam.stl"
@@ -199,5 +169,5 @@
         </visual>
         <collision>
-            <origin xyz="0.038 0 -0.0125" rpy="1.57 0 1.57" />
+            <origin xyz="0.038 0.0 -0.0125" rpy="1.57 0.0 1.57" />
             <geometry>
                 <mesh filename="package://aster_description/meshes/ownStls/Face_OLED_PiCam.stl"
@@ -228,5 +198,5 @@
     <link name="sh_rh_lift_link">
         <visual>
-            <origin xyz="0 0.108 -0.6625" rpy="0.0 0.0 0.0" />
+            <origin xyz="0.0 0.108 -0.6625" rpy="0.0 0.0 0.0" />
             <geometry>
                 <mesh filename="package://aster_description/meshes/Right_Arm_Shoulder.stl"
@@ -236,5 +206,5 @@
         </visual>
         <collision>
-            <origin xyz="0 0.108 -0.6625" rpy="0.0 0.0 0.0" />
+            <origin xyz="0.0 0.108 -0.6625" rpy="0.0 0.0 0.0" />
             <geometry>
                 <mesh filename="package://aster_description/meshes/Right_Arm_Shoulder.stl"
@@ -246,5 +216,5 @@
     <link name="sh_rh_rotate_link">
         <visual>
-            <origin xyz="0 0.108 0.51" rpy="${PI} 0 ${PI}" />
+            <origin xyz="0.0 0.108 0.51" rpy="${PI} 0.0 ${PI}" />
             <geometry>
                 <mesh filename="package://aster_description/meshes/Right_Arm_Upper.stl"
@@ -254,5 +224,5 @@
         </visual>
         <collision>
-            <origin xyz="0 0.108 0.51" rpy="${PI} 0 ${PI}" />
+            <origin xyz="0.0 0.108 0.51" rpy="${PI} 0.0 ${PI}" />
             <geometry>
                 <mesh filename="package://aster_description/meshes/Right_Arm_Upper.stl"
@@ -264,5 +234,5 @@
     <link name="elbow_rh_link">
         <visual>
-            <origin xyz="-0.01 0.1075 -0.498" rpy="0 0 0" />
+            <origin xyz="-0.01 0.1075 -0.498" rpy="0.0 0.0 0.0" />
             <geometry>
                 <mesh filename="package://aster_description/meshes/Right_Arm_Lower.stl"
@@ -272,5 +242,5 @@
         </visual>
         <collision>
-            <origin xyz="-0.01 0.1075 -0.498" rpy="0 0 0" />
+            <origin xyz="-0.01 0.1075 -0.498" rpy="0.0 0.0 0.0" />
             <geometry>
                 <mesh filename="package://aster_description/meshes/Right_Arm_Lower.stl"
@@ -282,5 +252,5 @@
     <link name="rh_rotate_link">
         <visual>
-            <origin xyz="-0.02 0 -0.03" rpy="${-PI/2} 0 ${-PI/2}" />
+            <origin xyz="-0.02 0.0 -0.03" rpy="${-PI/2} 0.0 ${-PI/2}" />
             <geometry>
                 <mesh
@@ -291,5 +261,5 @@
         </visual>
         <collision>
-            <origin xyz="-0.02 0 -0.03" rpy="${-PI/2} 0 ${-PI/2}" />
+            <origin xyz="-0.02 0.0 -0.03" rpy="${-PI/2} 0.0 ${-PI/2}" />
             <geometry>
                 <mesh
@@ -303,5 +273,5 @@
     <link name="rh_rotate_top_link" >
         <visual>
-            <origin xyz="-0.004 0 -0.03" rpy="${-PI/2} 0 ${-PI/2}"/>
+            <origin xyz="-0.004 0.0 -0.03" rpy="${-PI/2} 0.0 ${-PI/2}"/>
             <geometry>
                 <mesh filename="package://aster_description/meshes/Greifer/files/Robotic_Arm_Palm_Top.stl"
@@ -311,5 +281,5 @@
         </visual>
         <collision>
-            <origin xyz="-0.004 0 -0.03" rpy="${-PI/2} 0 ${-PI/2}"/>
+            <origin xyz="-0.004 0.0 -0.03" rpy="${-PI/2} 0.0 ${-PI/2}"/>
             <geometry>
                 <mesh filename="package://aster_description/meshes/Greifer/files/Robotic_Arm_Palm_Top.stl"
@@ -321,5 +291,5 @@
     <link name="rh_gripper1_link" >
         <visual>
-            <origin xyz="-0.005 0.016 -0.008" rpy="${-PI/2} 0 ${-PI/2}"/>
+            <origin xyz="-0.005 0.016 -0.008" rpy="${-PI/2} 0.0 ${-PI/2}"/>
             <geometry>
                 <mesh filename="package://aster_description/meshes/Greifer/files/Robotic_Arm_Finger.stl"
@@ -329,5 +299,5 @@
         </visual>
         <collision>
-            <origin xyz="-0.005 0.016 -0.008" rpy="${-PI/2} 0 ${-PI/2}"/>
+            <origin xyz="-0.005 0.016 -0.008" rpy="${-PI/2} 0.0 ${-PI/2}"/>
             <geometry>
                 <mesh filename="package://aster_description/meshes/Greifer/files/Robotic_Arm_Finger.stl"
@@ -339,5 +309,5 @@
     <link name="rh_gripper2_link" >
         <visual>
-            <origin xyz="0.007 -0.016 -0.008" rpy="${-PI/2} 0 ${PI/2}"/>
+            <origin xyz="0.007 -0.016 -0.008" rpy="${-PI/2} 0.0 ${PI/2}"/>
             <geometry>
                 <mesh filename="package://aster_description/meshes/Greifer/files/Robotic_Arm_Finger.stl"
@@ -347,5 +317,5 @@
         </visual>
         <collision>
-            <origin xyz="0.007 -0.016 -0.008" rpy="${-PI/2} 0 ${PI/2}"/>
+            <origin xyz="0.007 -0.016 -0.008" rpy="${-PI/2} 0.0 ${PI/2}"/>
             <geometry>
                 <mesh filename="package://aster_description/meshes/Greifer/files/Robotic_Arm_Finger.stl"
@@ -357,5 +327,5 @@
     <link name="rh_gripper1_pad_link" >
         <visual>
-            <origin xyz="-0.004 -0.0015 -0.0017" rpy="0 ${PI/2} 0"/>
+            <origin xyz="-0.004 -0.0015 -0.0017" rpy="0.0 ${PI/2} 0.0"/>
             <geometry>
                 <mesh filename="package://aster_description/meshes/Greifer/files/Robotic_Arm_Finger_Pad.stl"
@@ -365,5 +335,5 @@
         </visual>
         <collision>
-            <origin xyz="-0.004 -0.0015 -0.0017" rpy="0 ${PI/2} 0"/>
+            <origin xyz="-0.004 -0.0015 -0.0017" rpy="0.0 ${PI/2} 0.0"/>
             <geometry>
                 <mesh filename="package://aster_description/meshes/Greifer/files/Robotic_Arm_Finger_Pad.stl"
@@ -375,5 +345,5 @@
     <link name="rh_gripper2_pad_link" >
         <visual>
-            <origin xyz="0.005 0.0015 -0.0017" rpy="${PI} ${PI/2} 0"/>
+            <origin xyz="0.005 0.0015 -0.0017" rpy="${PI} ${PI/2} 0.0"/>
             <geometry>
                 <mesh filename="package://aster_description/meshes/Greifer/files/Robotic_Arm_Finger_Pad.stl"
@@ -383,5 +353,5 @@
         </visual>
         <collision>
-            <origin xyz="0.005 0.0015 -0.0017" rpy="${PI} ${PI/2} 0"/>
+            <origin xyz="0.005 0.0015 -0.0017" rpy="${PI} ${PI/2} 0.0"/>
             <geometry>
                 <mesh filename="package://aster_description/meshes/Greifer/files/Robotic_Arm_Finger_Pad.stl"
@@ -412,5 +382,5 @@
     <link name="sh_lh_lift_link">
         <visual>
-            <origin xyz="0 0 -0.036" rpy="0.0 0.0 0.0"/>
+            <origin xyz="0.0 0.0 -0.036" rpy="0.0 0.0 0.0"/>
             <geometry>
                 <mesh filename="package://aster_description/meshes/Left_Arm_Shoulder.stl" scale="0.001 0.001
@@ -420,5 +390,5 @@
         </visual>
         <collision>
-            <origin xyz="0 0 -0.036" rpy="0.0 0.0 0.0"/>
+            <origin xyz="0.0 0.0 -0.036" rpy="0.0 0.0 0.0"/>
             <geometry>
                 <mesh filename="package://aster_description/meshes/Left_Arm_Shoulder.stl" scale="0.001 0.001
@@ -430,5 +400,5 @@
     <link name="sh_lh_rotate_link">
         <visual>
-            <origin xyz="0 0 -0.005" rpy="${PI} 0 ${PI}"/>
+            <origin xyz="0.0 0.0 -0.005" rpy="${PI} 0.0 ${PI}"/>
             <geometry>
                 <mesh filename="package://aster_description/meshes/Left_Arm_Upper.stl" scale="0.001 0.001 0.001"/>
@@ -437,5 +407,5 @@
         </visual>
         <collision>
-            <origin xyz="0 0 -0.005" rpy="${PI} 0 ${PI}"/>
+            <origin xyz="0.0 0.0 -0.005" rpy="${PI} 0.0 ${PI}"/>
             <geometry>
                 <mesh filename="package://aster_description/meshes/Left_Arm_Upper.stl" scale="0.001 0.001 0.001"/>
@@ -446,5 +416,5 @@
     <link name="elbow_lh_link">
         <visual>
-            <origin xyz="-0.06 0.002 -0.008" rpy="0 0 0"/>
+            <origin xyz="-0.06 0.002 -0.008" rpy="0.0 0.0 0.0"/>
             <geometry>
                 <mesh filename="package://aster_description/meshes/Left_Arm_Lower.stl" scale="0.001 0.001 0.001"/>
@@ -453,5 +423,5 @@
         </visual>
         <collision>
-            <origin xyz="-0.06 0.002 -0.008" rpy="0 0 0"/>
+            <origin xyz="-0.06 0.002 -0.008" rpy="0.0 0.0 0.0"/>
             <geometry>
                 <mesh filename="package://aster_description/meshes/Left_Arm_Lower.stl" scale="0.001 0.001 0.001"/>
@@ -462,5 +432,5 @@
     <link name="lh_rotate_link" >
         <visual>
-            <origin xyz="-0.02 0 -0.03" rpy="${-PI/2} 0 ${-PI/2}"/>
+            <origin xyz="-0.02 0.0 -0.03" rpy="${-PI/2} 0.0 ${-PI/2}"/>
             <geometry>
                 <mesh filename="package://aster_description/meshes/Greifer/files/Robotic_Arm_Palm.stl" scale="0.001
@@ -470,5 +440,5 @@
         </visual>
         <collision>
-            <origin xyz="-0.02 0 -0.03" rpy="${-PI/2} 0 ${-PI/2}"/>
+            <origin xyz="-0.02 0.0 -0.03" rpy="${-PI/2} 0.0 ${-PI/2}"/>
             <geometry>
                 <mesh filename="package://aster_description/meshes/Greifer/files/Robotic_Arm_Palm.stl" scale="0.001
@@ -481,5 +451,5 @@
     <link name="lh_rotate_top_link" >
         <visual>
-            <origin xyz="-0.004 0 -0.03" rpy="${-PI/2} 0 ${-PI/2}"/>
+            <origin xyz="-0.004 0.0 -0.03" rpy="${-PI/2} 0.0 ${-PI/2}"/>
             <geometry>
                 <mesh filename="package://aster_description/meshes/Greifer/files/Robotic_Arm_Palm_Top.stl"
@@ -489,5 +459,5 @@
         </visual>
         <collision>
-            <origin xyz="-0.004 0 -0.03" rpy="${-PI/2} 0 ${-PI/2}"/>
+            <origin xyz="-0.004 0.0 -0.03" rpy="${-PI/2} 0.0 ${-PI/2}"/>
             <geometry>
                 <mesh filename="package://aster_description/meshes/Greifer/files/Robotic_Arm_Palm_Top.stl"
@@ -499,5 +469,5 @@
     <link name="lh_gripper1_link" >
         <visual>
-            <origin xyz="-0.005 0.016 -0.008" rpy="${-PI/2} 0 ${-PI/2}"/>
+            <origin xyz="-0.005 0.016 -0.008" rpy="${-PI/2} 0.0 ${-PI/2}"/>
             <geometry>
                 <mesh filename="package://aster_description/meshes/Greifer/files/Robotic_Arm_Finger.stl"
@@ -507,5 +477,5 @@
         </visual>
         <collision>
-            <origin xyz="-0.005 0.016 -0.008" rpy="${-PI/2} 0 ${-PI/2}"/>
+            <origin xyz="-0.005 0.016 -0.008" rpy="${-PI/2} 0.0 ${-PI/2}"/>
             <geometry>
                 <mesh filename="package://aster_description/meshes/Greifer/files/Robotic_Arm_Finger.stl"
@@ -517,5 +487,5 @@
     <link name="lh_gripper2_link" >
         <visual>
-            <origin xyz="0.007 -0.016 -0.008" rpy="${-PI/2} 0 ${PI/2}"/>
+            <origin xyz="0.007 -0.016 -0.008" rpy="${-PI/2} 0.0 ${PI/2}"/>
             <geometry>
                 <mesh filename="package://aster_description/meshes/Greifer/files/Robotic_Arm_Finger.stl"
@@ -525,5 +495,5 @@
         </visual>
         <collision>
-            <origin xyz="0.007 -0.016 -0.008" rpy="${-PI/2} 0 ${PI/2}"/>
+            <origin xyz="0.007 -0.016 -0.008" rpy="${-PI/2} 0.0 ${PI/2}"/>
             <geometry>
                 <mesh filename="package://aster_description/meshes/Greifer/files/Robotic_Arm_Finger.stl"
@@ -535,5 +505,5 @@
     <link name="lh_gripper1_pad_link" >
         <visual>
-            <origin xyz="-0.004 -0.0015 -0.0017" rpy="0 ${PI/2} 0"/>
+            <origin xyz="-0.004 -0.0015 -0.0017" rpy="0.0 ${PI/2} 0.0"/>
             <geometry>
                 <mesh filename="package://aster_description/meshes/Greifer/files/Robotic_Arm_Finger_Pad.stl"
@@ -543,5 +513,5 @@
         </visual>
         <collision>
-            <origin xyz="-0.004 -0.0015 -0.0017" rpy="0 ${PI/2} 0"/>
+            <origin xyz="-0.004 -0.0015 -0.0017" rpy="0.0 ${PI/2} 0.0"/>
             <geometry>
                 <mesh filename="package://aster_description/meshes/Greifer/files/Robotic_Arm_Finger_Pad.stl"
@@ -553,5 +523,5 @@
     <link name="lh_gripper2_pad_link" >
         <visual>
-            <origin xyz="0.005 0.0015 -0.0017" rpy="${PI} ${PI/2} 0"/>
+            <origin xyz="0.005 0.0015 -0.0017" rpy="${PI} ${PI/2} 0.0"/>
             <geometry>
                 <mesh filename="package://aster_description/meshes/Greifer/files/Robotic_Arm_Finger_Pad.stl"
@@ -561,5 +531,5 @@
         </visual>
         <collision>
-            <origin xyz="0.005 0.0015 -0.0017" rpy="${PI} ${PI/2} 0"/>
+            <origin xyz="0.005 0.0015 -0.0017" rpy="${PI} ${PI/2} 0.0"/>
             <geometry>
                 <mesh filename="package://aster_description/meshes/Greifer/files/Robotic_Arm_Finger_Pad.stl"
@@ -572,5 +542,5 @@
     <link name="hip_rh_link">
         <visual>
-            <origin xyz="0.0023 -0.015 -0.1748" rpy="0 0 0"/>
+            <origin xyz="0.0023 -0.015 -0.1748" rpy="0.0 0.0 0.0"/>
             <geometry>
                 <mesh filename="package://aster_description/meshes/Right_Leg_Upper.stl" scale="0.001 0.001 0.001"/>
@@ -579,5 +549,5 @@
         </visual>
         <collision>
-            <origin xyz="0.0023 -0.015 -0.1748" rpy="0 0 0"/>
+            <origin xyz="0.0023 -0.015 -0.1748" rpy="0.0 0.0 0.0"/>
             <geometry>
                 <mesh filename="package://aster_description/meshes/Right_Leg_Upper.stl" scale="0.001 0.001 0.001"/>
@@ -588,5 +558,5 @@
     <link name="knie_rh_link" >
         <visual>
-            <origin xyz="0.0025 0 -0.1765" rpy="0 0 0"/>
+            <origin xyz="0.0025 0.0 -0.1765" rpy="0.0 0.0 0.0"/>
             <geometry>
                 <mesh filename="package://aster_description/meshes/Right_Leg_Lower.stl" scale="0.001 0.001 0.001"/>
@@ -595,5 +565,5 @@
         </visual>
         <collision>
-            <origin xyz="0.0025 0 -0.1765" rpy="0 0 0"/>
+            <origin xyz="0.0025 0.0 -0.1765" rpy="0.0 0.0 0.0"/>
             <geometry>
                 <mesh filename="package://aster_description/meshes/Right_Leg_Lower.stl" scale="0.001 0.001 0.001"/>
@@ -604,5 +574,5 @@
     <link name="foot_rh_link" >
         <visual>
-            <origin xyz="0.03 -0.0025 -0.035" rpy="0 0 0"/>
+            <origin xyz="0.03 -0.0025 -0.035" rpy="0.0 0.0 0.0"/>
             <geometry>
                 <mesh filename="package://aster_description/meshes/Right_Leg_Foot.stl" scale="0.001 0.001 0.001"/>
@@ -611,5 +581,5 @@
         </visual>
         <collision>
-            <origin xyz="0.03 -0.0025 -0.035" rpy="0 0 0"/>
+            <origin xyz="0.03 -0.0025 -0.035" rpy="0.0 0.0 0.0"/>
             <geometry>
                 <mesh filename="package://aster_description/meshes/Right_Leg_Foot.stl" scale="0.001 0.001 0.001"/>
@@ -621,5 +591,5 @@
     <link name="hip_lh_link">
         <visual>
-            <origin xyz="0.0023 0.015 -0.1748" rpy="0 0 0"/>
+            <origin xyz="0.0023 0.015 -0.1748" rpy="0.0 0.0 0.0"/>
             <geometry>
                 <mesh filename="package://aster_description/meshes/Left_Leg_Upper.stl" scale="0.001 0.001 0.001"/>
@@ -628,5 +598,5 @@
         </visual>
         <collision>
-            <origin xyz="0.0023 0.015 -0.1748" rpy="0 0 0"/>
+            <origin xyz="0.0023 0.015 -0.1748" rpy="0.0 0.0 0.0"/>
             <geometry>
                 <mesh filename="package://aster_description/meshes/Left_Leg_Upper.stl" scale="0.001 0.001 0.001"/>
@@ -637,5 +607,5 @@
     <link name="knie_lh_link" >
         <visual>
-            <origin xyz="0.0025 0 -0.1765" rpy="0 0 0"/>
+            <origin xyz="0.0025 0.0 -0.1765" rpy="0.0 0.0 0.0"/>
             <geometry>
                 <mesh filename="package://aster_description/meshes/Left_Lower_Leg.stl" scale="0.001 0.001 0.001"/>
@@ -644,5 +614,5 @@
         </visual>
         <collision>
-            <origin xyz="0.0025 0 -0.1765" rpy="0 0 0"/>
+            <origin xyz="0.0025 0.0 -0.1765" rpy="0.0 0.0 0.0"/>
             <geometry>
                 <mesh filename="package://aster_description/meshes/Left_Lower_Leg.stl" scale="0.001 0.001 0.001"/>
@@ -653,5 +623,5 @@
     <link name="foot_lh_link" >
         <visual>
-            <origin xyz="0.03 0.0025 -0.035" rpy="0 0 0"/>
+            <origin xyz="0.03 0.0025 -0.035" rpy="0.0 0.0 0.0"/>
             <geometry>
                 <mesh filename="package://aster_description/meshes/Left_Leg_Foot.stl" scale="0.001 0.001 0.001"/>
@@ -660,5 +630,5 @@
         </visual>
         <collision>
-            <origin xyz="0.03 0.0025 -0.035" rpy="0 0 0"/>
+            <origin xyz="0.03 0.0025 -0.035" rpy="0.0 0.0 0.0"/>
             <geometry>
                 <mesh filename="package://aster_description/meshes/Left_Leg_Foot.stl" scale="0.001 0.001 0.001"/>
@@ -687,15 +657,15 @@
         <parent link="chest_bone_link" />
         <child link="chest_link" />
-        <origin xyz="0 0 0" rpy="0.0 0.0 0.0" />
+        <origin xyz="0.0 0.0 0.0" rpy="0.0 0.0 0.0" />
     </joint>
     <joint name="chestbone_to_backbone" type="fixed">
         <parent link="chest_bone_link" />
         <child link="backbone_link" />
-        <origin xyz="0 0 0" rpy="0.0 0.0 0.0" />
+        <origin xyz="0.0 0.0 0.0" rpy="0.0 0.0 0.0" />
     </joint>
     <joint name="backbone_to_hip" type="fixed">
         <parent link="backbone_link" />
         <child link="hip_link" />
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
File: aster_description/urdf/gazebo.xacro (robot description, xacro)
@@ -1,11 +1,39 @@
 <?xml version="1.0"?>
-<robot xmlns:xacro="http://www.ros.org/wiki/xacro" name="aster">
-    <!-- Gazebo ros2_control plugin -->
+<robot xmlns:xacro="http://www.ros.org/wiki/xacro" name="rca">
     <gazebo>
-      <plugin filename="libgazebo_ros2_control.so" name="gazebo_ros2_control">
-        <robot_param>robot_description</robot_param>
-        <robot_param_node>robot_state_publisher</robot_param_node>
-        <parameters>$(find aster_controller)/config/controllers.yaml</parameters>
-      </plugin>
+        <plugin filename="libgazebo_ros2_control.so" name="gazebo_ros2_control">
+            <robot_param>robot_description</robot_param>
+            <robot_param_node>robot_state_publisher</robot_param_node>
+            <parameters>$(find aster_controller)/config/aster_controllers.yaml</parameters>
+        </plugin>
     </gazebo>
+<!--
+    <gazebo reference="base_link">
+        <material>Gazebo/Black</material>
+    </gazebo>
+    <gazebo reference="base_holder_link">
+        <material>Gazebo/Blue</material>
+    </gazebo>
+    <gazebo reference="chest_bone_link">
+        <material>Gazebo/White</material>
+    </gazebo>
+    <gazebo reference="chest_link">
+        <material>Gazebo/White</material>
+    </gazebo>
+    <gazebo reference="backbone_link">
+        <material>Gazebo/White</material>
+    </gazebo>
+    <gazebo reference="hip_link">
+        <material>Gazebo/Black</material>
+    </gazebo>
+    <gazebo reference="neck_link">
+        <material>Gazebo/Green</material>
+    </gazebo>
+    <gazebo reference="head_link">
+        <material>Gazebo/Red</material>
+    </gazebo>
+    <gazebo reference="face_link">
+        <material>Gazebo/Black</material>
+    </gazebo>
+    -->
 </robot>
