Commit message: gazebo and controllers

File: aster_description/urdf/aster.urdf.xacro (robot description, xacro)
@@ -3,3 +3,4 @@
     <xacro:include filename="material.xacro"/>
     <xacro:include filename="aster.xacro"/>
+    <xacro:include filename="aster_gazebo.xacro"/>
 </robot>

File: aster_description/urdf/aster.xacro (robot description, xacro)
@@ -2,4 +2,14 @@
 <robot xmlns:xacro="http://www.ros.org/wiki/xacro" >
     <!-- <xacro:default_inertial mass="0.3"/> -->
+    <!-- <xacro:default_inertial_1 mass="0.03"/> -->
+    <xacro:macro name="default_transmission" params="number">
+        <transmission name="transmission_${number}">
+            <plugin>transmission_interface/SimpleTransmission</plugin>
+            <actuator name="motor_${number}" role="actuator1"/>
+            <joint name="joint_${number}"    role="joint1">
+                <mechanical_reduction>1.0</mechanical_reduction>
+            </joint>
+        </transmission>
+    </xacro:macro>
     <link name="world"/>
     <link name="base_link">
@@ -11,4 +21,11 @@
             <material name="white"/>
         </visual>
+        <collision>
+            <origin xyz="0.0 0.0 0.0" rpy="0.0 0.0 0.0"/>
+            <geometry>
+                <mesh filename="package://aster_description/meshes/ownStls/standBase.stl" scale="0.001 0.001 0.001"/>
+            </geometry>
+        </collision>
+        <xacro:default_inertial mass="3.3"/>
     </link>
     <!-- Base-->
@@ -21,4 +38,11 @@
             <material name="white"/>
         </visual>
+        <collision>
+            <origin xyz="0.0 0.0 -0.02" rpy="0.0 0.0 ${-PI/2}"/>
+            <geometry>
+                <mesh filename="package://aster_description/meshes/subStuff/RohrHalter_v2.stl" scale="0.001 0.001 0.001"/>
+            </geometry>
+        </collision>
+        <xacro:default_inertial mass="0.3"/>
     </link>
     <link name="chest_bone_link">
@@ -30,4 +54,11 @@
             <material name="white"/>
         </visual>
+        <collision>
+            <origin xyz="0.0 0.0 0.0" rpy="0.0 0.0 0.0"/>
+            <geometry>
+                <mesh filename="package://aster_description/meshes/Spine_Connector.stl" scale="0.001 0.001 0.001"/>
+            </geometry>
+        </collision>
+        <xacro:default_inertial mass="0.3"/>
     </link>
     <link name="chest_link">
@@ -39,4 +70,11 @@
             <material name="black"/>
         </visual>
+        <collision>
+            <origin xyz="0.0 0.0 -0.012" rpy="0.0 0.0 0.0"/>
+            <geometry>
+                <mesh filename="package://aster_description/meshes/Chest.stl" scale="0.001 0.001 0.001"/>
+            </geometry>
+        </collision>
+        <xacro:default_inertial mass="0.3"/>
     </link>
     <link name="backbone_link">
@@ -48,4 +86,11 @@
             <material name="white"/>
         </visual>
+        <collision>
+            <origin xyz="-0.003 0.0 -0.085" rpy="0.0 0.0 0.0"/>
+            <geometry>
+                <mesh filename="package://aster_description/meshes/Spine.stl" scale="0.001 0.001 0.001"/>
+            </geometry>
+        </collision>
+        <xacro:default_inertial mass="0.3"/>
     </link>
     <link name="hip_link">
@@ -57,4 +102,11 @@
             <material name="white"/>
         </visual>
+        <collision>
+            <origin xyz="-0.005 0.0 0.003" rpy="0.0 0.0 0.0"/>
+            <geometry>
+                <mesh filename="package://aster_description/meshes/Hips.stl" scale="0.001 0.001 0.001"/>
+            </geometry>
+        </collision>
+        <xacro:default_inertial mass="0.3"/>
     </link>
    <!-- Head-->
@@ -67,4 +119,11 @@
             <material name="blue"/>
         </visual>
+        <collision>
+            <origin xyz="0.0 0.0 -0.012" rpy="0.0 0.0 0.0"/>
+            <geometry>
+                <mesh filename="package://aster_description/meshes/Head_Neck.stl" scale="0.001 0.001 0.001"/>
+            </geometry>
+        </collision>
+        <xacro:default_inertial mass="0.3"/>
     </link>
     <link name="head_link">
@@ -76,4 +135,11 @@
             <material name="white"/>
         </visual>
+        <collision>
+            <origin xyz="0.0 0.0 -0.012" rpy="0.0 0.0 0.0"/>
+            <geometry>
+                <mesh filename="package://aster_description/meshes/Head_Back.stl" scale="0.001 0.001 0.001"/>
+            </geometry>
+        </collision>
+        <xacro:default_inertial mass="0.3"/>
     </link>
     <link name="face_link">
@@ -85,4 +151,11 @@
             <material name="black"/>
         </visual>
+        <collision>
+            <origin xyz="0.038 0 -0.0125" rpy="1.57 0 1.57"/>
+            <geometry>
+                <mesh filename="package://aster_description/meshes/ownStls/Face_OLED_PiCam.stl" scale="0.001 0.001 0.001"/>
+            </geometry>
+        </collision>
+        <xacro:default_inertial mass="0.3"/>
     </link>
     <!-- Right Arm-->
@@ -95,4 +168,11 @@
             <material name="white"/>
         </visual>
+        <collision>
+            <origin xyz="-0.01 -0.018 -0.023" rpy="0.0 0.0 0.0"/>
+            <geometry>
+                <mesh filename="package://aster_description/meshes/Rigth_Arm_Shoulder_Connector.stl" scale="0.001 0.001 0.001"/>
+            </geometry>
+        </collision>
+        <xacro:default_inertial mass="0.3"/>
     </link>
     <link name="sh_rh_lift_link">
@@ -104,4 +184,11 @@
             <material name="white"/>
         </visual>
+        <collision>
+            <origin xyz="0 0.108 -0.6625" rpy="0.0 0.0 0.0"/>
+            <geometry>
+                <mesh filename="package://aster_description/meshes/Right_Arm_Shoulder.stl" scale="0.001 0.001 0.001"/>
+            </geometry>
+        </collision>
+        <xacro:default_inertial mass="0.3"/>
     </link>
     <link name="sh_rh_rotate_link">
@@ -113,4 +200,11 @@
             <material name="white"/>
         </visual>
+        <collision>
+            <origin xyz="0 0.108 0.51" rpy="${PI} 0 ${PI}"/>
+            <geometry>
+                <mesh filename="package://aster_description/meshes/Right_Arm_Upper.stl" scale="0.001 0.001 0.001"/>
+            </geometry>
+        </collision>
+        <xacro:default_inertial mass="0.3"/>
     </link>
     <link name="elbow_rh_link">
@@ -122,15 +216,29 @@
             <material name="white"/>
         </visual>
+        <collision>
+            <origin xyz="-0.01 0.1075 -0.498" rpy="0 0 0"/>
+            <geometry>
+                <mesh filename="package://aster_description/meshes/Right_Arm_Lower.stl" scale="0.001 0.001 0.001"/>
+            </geometry>
+        </collision>
+        <xacro:default_inertial mass="0.3"/>
+    </link>
+    <link name="rh_rotate_link" >
+        <visual>
+            <origin xyz="-0.02 0 -0.03" rpy="${-PI/2} 0 ${-PI/2}"/>
+            <geometry>
+                <mesh filename="package://aster_description/meshes/Greifer/files/Robotic_Arm_Palm.stl" scale="0.001 0.001 0.001"/>
+            </geometry>
+            <material name="white"/>
+        </visual>
+        <collision>
+            <origin xyz="-0.02 0 -0.03" rpy="${-PI/2} 0 ${-PI/2}"/>
+            <geometry>
+                <mesh filename="package://aster_description/meshes/Greifer/files/Robotic_Arm_Palm.stl" scale="0.001 0.001 0.001"/>
+            </geometry>
+        </collision>
+        <xacro:default_inertial mass="0.3"/>
     </link>
     <!-- Right Gripper-->
-    <link name="rh_rotate_link" >
-        <visual>
-            <origin xyz="-0.02 0 -0.03" rpy="${-PI/2} 0 ${-PI/2}"/>
-            <geometry>
-                <mesh filename="package://aster_description/meshes/Greifer/files/Robotic_Arm_Palm.stl" scale="0.001 0.001 0.001"/>
-            </geometry>
-            <material name="white"/>
-        </visual>
-    </link>
     <link name="rh_rotate_top_link" >
         <visual>
@@ -141,4 +249,11 @@
             <material name="white"/>
         </visual>
+        <collision>
+            <origin xyz="-0.004 0 -0.03" rpy="${-PI/2} 0 ${-PI/2}"/>
+            <geometry>
+                <mesh filename="package://aster_description/meshes/Greifer/files/Robotic_Arm_Palm_Top.stl" scale="0.001 0.001 0.001"/>
+            </geometry>
+        </collision>
+        <xacro:default_inertial mass="0.3"/>
     </link>
     <link name="rh_gripper1_link" >
@@ -150,4 +265,11 @@
             <material name="white"/>
         </visual>
+        <collision>
+            <origin xyz="-0.005 0.016 -0.008" rpy="${-PI/2} 0 ${-PI/2}"/>
+            <geometry>
+                <mesh filename="package://aster_description/meshes/Greifer/files/Robotic_Arm_Finger.stl" scale="0.001 0.001 0.001"/>
+            </geometry>
+        </collision>
+        <xacro:default_inertial mass="0.3"/>
     </link>
     <link name="rh_gripper2_link" >
@@ -159,4 +281,11 @@
             <material name="white"/>
         </visual>
+        <collision>
+            <origin xyz="0.007 -0.016 -0.008" rpy="${-PI/2} 0 ${PI/2}"/>
+            <geometry>
+                <mesh filename="package://aster_description/meshes/Greifer/files/Robotic_Arm_Finger.stl" scale="0.001 0.001 0.001"/>
+            </geometry>
+        </collision>
+        <xacro:default_inertial mass="0.3"/>
     </link>
     <link name="rh_gripper1_pad_link" >
@@ -168,4 +297,11 @@
             <material name="black"/>
         </visual>
+        <collision>
+            <origin xyz="-0.004 -0.0015 -0.0017" rpy="0 ${PI/2} 0"/>
+            <geometry>
+                <mesh filename="package://aster_description/meshes/Greifer/files/Robotic_Arm_Finger_Pad.stl" scale="0.001 0.001 0.001"/>
+            </geometry>
+        </collision>
+        <xacro:default_inertial_1 mass="0.03"/>
     </link>
     <link name="rh_gripper2_pad_link" >
@@ -177,4 +313,11 @@
             <material name="black"/>
         </visual>
+        <collision>
+            <origin xyz="0.005 0.0015 -0.0017" rpy="${PI} ${PI/2} 0"/>
+            <geometry>
+                <mesh filename="package://aster_description/meshes/Greifer/files/Robotic_Arm_Finger_Pad.stl" scale="0.001 0.001 0.001"/>
+            </geometry>
+        </collision>
+        <xacro:default_inertial_1 mass="0.03"/>
     </link>
     <!-- Left Arm-->
@@ -187,4 +330,11 @@
             <material name="white"/>
         </visual>
+        <collision>
+            <origin xyz="-0.01 0.018 -0.023" rpy="0.0 0.0 0.0"/>
+            <geometry>
+                <mesh filename="package://aster_description/meshes/Left_Arm_Shoulder_Connector.stl" scale="0.001 0.001 0.001"/>
+            </geometry>
+        </collision>
+        <xacro:default_inertial mass="0.3"/>
     </link>
     <link name="sh_lh_lift_link">
@@ -196,4 +346,11 @@
             <material name="white"/>
         </visual>
+        <collision>
+            <origin xyz="0 0 -0.036" rpy="0.0 0.0 0.0"/>
+            <geometry>
+                <mesh filename="package://aster_description/meshes/Left_Arm_Shoulder.stl" scale="0.001 0.001 0.001"/>
+            </geometry>
+        </collision>
+        <xacro:default_inertial mass="0.3"/>
     </link>
     <link name="sh_lh_rotate_link">
@@ -205,4 +362,11 @@
             <material name="white"/>
         </visual>
+        <collision>
+            <origin xyz="0 0 -0.005" rpy="${PI} 0 ${PI}"/>
+            <geometry>
+                <mesh filename="package://aster_description/meshes/Left_Arm_Upper.stl" scale="0.001 0.001 0.001"/>
+            </geometry>
+        </collision>
+        <xacro:default_inertial mass="0.3"/>
     </link>
     <link name="elbow_lh_link">
@@ -214,15 +378,29 @@
             <material name="white"/>
         </visual>
+        <collision>
+            <origin xyz="-0.06 0.002 -0.008" rpy="0 0 0"/>
+            <geometry>
+                <mesh filename="package://aster_description/meshes/Left_Arm_Lower.stl" scale="0.001 0.001 0.001"/>
+            </geometry>
+        </collision>
+        <xacro:default_inertial mass="0.3"/>
+    </link>
+    <link name="lh_rotate_link" >
+        <visual>
+            <origin xyz="-0.02 0 -0.03" rpy="${-PI/2} 0 ${-PI/2}"/>
+            <geometry>
+                <mesh filename="package://aster_description/meshes/Greifer/files/Robotic_Arm_Palm.stl" scale="0.001 0.001 0.001"/>
+            </geometry>
+            <material name="white"/>
+        </visual>
+        <collision>
+            <origin xyz="-0.02 0 -0.03" rpy="${-PI/2} 0 ${-PI/2}"/>
+            <geometry>
+                <mesh filename="package://aster_description/meshes/Greifer/files/Robotic_Arm_Palm.stl" scale="0.001 0.001 0.001"/>
+            </geometry>
+        </collision>
+        <xacro:default_inertial mass="0.3"/>
     </link>
     <!-- Left Gripper-->
-    <link name="lh_rotate_link" >
-        <visual>
-            <origin xyz="-0.02 0 -0.03" rpy="${-PI/2} 0 ${-PI/2}"/>
-            <geometry>
-                <mesh filename="package://aster_description/meshes/Greifer/files/Robotic_Arm_Palm.stl" scale="0.001 0.001 0.001"/>
-            </geometry>
-            <material name="white"/>
-        </visual>
-    </link>
     <link name="lh_rotate_top_link" >
         <visual>
@@ -233,4 +411,11 @@
             <material name="white"/>
         </visual>
+        <collision>
+            <origin xyz="-0.004 0 -0.03" rpy="${-PI/2} 0 ${-PI/2}"/>
+            <geometry>
+                <mesh filename="package://aster_description/meshes/Greifer/files/Robotic_Arm_Palm_Top.stl" scale="0.001 0.001 0.001"/>
+            </geometry>
+        </collision>
+        <xacro:default_inertial mass="0.3"/>
     </link>
     <link name="lh_gripper1_link" >
@@ -242,4 +427,11 @@
             <material name="white"/>
         </visual>
+        <collision>
+            <origin xyz="-0.005 0.016 -0.008" rpy="${-PI/2} 0 ${-PI/2}"/>
+            <geometry>
+                <mesh filename="package://aster_description/meshes/Greifer/files/Robotic_Arm_Finger.stl" scale="0.001 0.001 0.001"/>
+            </geometry>
+        </collision>
+        <xacro:default_inertial mass="0.3"/>
     </link>
     <link name="lh_gripper2_link" >
@@ -251,4 +443,11 @@
             <material name="white"/>
         </visual>
+        <collision>
+            <origin xyz="0.007 -0.016 -0.008" rpy="${-PI/2} 0 ${PI/2}"/>
+            <geometry>
+                <mesh filename="package://aster_description/meshes/Greifer/files/Robotic_Arm_Finger.stl" scale="0.001 0.001 0.001"/>
+            </geometry>
+        </collision>
+        <xacro:default_inertial mass="0.3"/>
     </link>
     <link name="lh_gripper1_pad_link" >
@@ -260,4 +459,11 @@
             <material name="black"/>
         </visual>
+        <collision>
+            <origin xyz="-0.004 -0.0015 -0.0017" rpy="0 ${PI/2} 0"/>
+            <geometry>
+                <mesh filename="package://aster_description/meshes/Greifer/files/Robotic_Arm_Finger_Pad.stl" scale="0.001 0.001 0.001"/>
+            </geometry>
+        </collision>
+        <xacro:default_inertial mass="0.3"/>
     </link>
     <link name="lh_gripper2_pad_link" >
@@ -269,4 +475,11 @@
             <material name="black"/>
         </visual>
+        <collision>
+            <origin xyz="0.005 0.0015 -0.0017" rpy="${PI} ${PI/2} 0"/>
+            <geometry>
+                <mesh filename="package://aster_description/meshes/Greifer/files/Robotic_Arm_Finger_Pad.stl" scale="0.001 0.001 0.001"/>
+            </geometry>
+        </collision>
+        <xacro:default_inertial mass="0.3"/>
     </link>
     <!-- Right Leg-->
@@ -279,4 +492,11 @@
             <material name="white"/>
         </visual>
+        <collision>
+            <origin xyz="0.0023 -0.015 -0.1748" rpy="0 0 0"/>
+            <geometry>
+                <mesh filename="package://aster_description/meshes/Right_Leg_Upper.stl" scale="0.001 0.001 0.001"/>
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
File: aster_description/urdf/material.xacro (robot description, xacro)
@@ -22,3 +22,11 @@
         </inertial>
     </xacro:macro>
+    <xacro:macro name="default_inertial_1" params="mass"> <!-- <xacro:default_inertial_1 mass="1.0"/> -->
+        <inertial>
+            <mass value="${mass}" />
+            <inertia ixx="0.00001" ixy="0.0" ixz="0.0"
+                     iyy="0.00001" iyz="0.0"
+                     izz="0.00001" />
+        </inertial>
+    </xacro:macro>
 </robot>

Commit message: second run

File: aster_description/urdf/aster.urdf.xacro (robot description, xacro)
@@ -1,7 +1,9 @@
 <?xml version="1.0"?>
 <robot xmlns:xacro="http://www.ros.org/wiki/xacro" name="aster">
-    <xacro:include filename="material.xacro"/>
-    <xacro:include filename="aster.xacro"/>
-    <xacro:include filename="aster_gazebo.xacro"/>
-    <xacro:include filename="aster_ros2_control.xacro"/>
+    <xacro:include filename="$(find aster_description)/urdf/material.xacro"/>
+    <xacro:include filename="$(find aster_description)/urdf/aster.xacro"/>
+<!--
+    <xacro:include filename="$(find aster_description)/urdf/aster_gazebo.xacro"/>
+    <xacro:include filename="$(find aster_description)/urdf/aster_ros2_control.xacro"/>
+-->
 </robot>

File: aster_description/urdf/aster.xacro (robot description, xacro)
@@ -583,30 +583,30 @@
                     <!-- ######  JOINTS  ######-->
     <!-- Base Virtual Joints-->
-    <joint name="virtual_1_joint" type="fixed">
+    <joint name="world_to_base" type="fixed">
         <parent link="world"/>
         <child link="base_link"/>
         <origin xyz="0.0 0.0 0.0" rpy="0.0 0.0 0.0"/>
     </joint>
-    <joint name="virtual_2_joint" type="fixed">
+    <joint name="base_to_holder" type="fixed">
         <parent link="base_link"/>
         <child link="base_holder_link"/>
         <origin xyz="0.0 0.0 0.62" rpy="0.0 0.0 0.0"/>
     </joint>
-    <joint name="virtual_3_joint" type="fixed">
+    <joint name="baseholder_to_chestbone" type="fixed">
         <parent link="base_holder_link"/>
         <child link="chest_bone_link"/>
         <origin xyz="0.042 0.0 0.015" rpy="0.0 0.0 0.0"/>
     </joint>
-    <joint name="virtual_4_joint" type="fixed">
+    <joint name="chestbone_to_chest" type="fixed">
         <parent link="chest_bone_link"/>
         <child link="chest_link"/>
         <origin xyz="0 0 0" rpy="0.0 0.0 0.0"/>
     </joint>
-    <joint name="virtual_5_joint" type="fixed">
+    <joint name="chestbone_to_backbone" type="fixed">
         <parent link="chest_bone_link"/>
         <child link="backbone_link"/>
         <origin xyz="0 0 0" rpy="0.0 0.0 0.0"/>
     </joint>
-    <joint name="virtual_6_joint" type="fixed">
+    <joint name="backbone_to_hip" type="fixed">
         <parent link="backbone_link"/>
         <child link="hip_link"/>
@@ -670,5 +670,5 @@
     </joint>
     <!-- Right Gripper Joints-->
-    <joint name="virtual_7_joint" type="fixed">
+    <joint name="gripper_body_rh" type="fixed">
         <parent link="rh_rotate_link"/>
         <child link="rh_rotate_top_link"/>
@@ -690,10 +690,10 @@
         <origin xyz="-0.015 0.02 -0.048" rpy="0 0 0"/>
     </joint>
-    <joint name="virtual_8_joint" type="fixed">
+    <joint name="pad_rh_r" type="fixed">
         <parent link="rh_gripper1_link"/>
         <child link="rh_gripper1_pad_link"/>
         <origin xyz="0 0.015 -0.041" rpy="0.0 0.0 0.0"/>
     </joint>
-    <joint name="virtual_9_joint" type="fixed">
+    <joint name="pad_rh_l" type="fixed">
         <parent link="rh_gripper2_link"/>
         <child link="rh_gripper2_pad_link"/>
@@ -737,5 +737,5 @@
     </joint>
     <!-- Left Gripper Joints-->
-    <joint name="virtual_10_joint" type="fixed">
+    <joint name="gripper_body_lh" type="fixed">
         <parent link="lh_rotate_link"/>
         <child link="lh_rotate_top_link"/>
@@ -757,10 +757,10 @@
         <origin xyz="-0.015 0.02 -0.048" rpy="0 0 0"/>
     </joint>
-    <joint name="virtual_11_joint" type="fixed">
+    <joint name="pad_lh_r" type="fixed">
         <parent link="lh_gripper1_link"/>
         <child link="lh_gripper1_pad_link"/>
         <origin xyz="0 0.015 -0.041" rpy="0.0 0.0 0.0"/>
     </joint>
-    <joint name="virtual_12_joint" type="fixed">
+    <joint name="pad_lh_l" type="fixed">
         <parent link="lh_gripper2_link"/>
         <child link="lh_gripper2_pad_link"/>

File: aster_description/urdf/aster_ros2_control.xacro (robot description, xacro)
@@ -1,4 +1,4 @@
 <?xml version="1.0"?>
-<robot xmlns:xacro="http://www.ros.org/wiki/xacro" name="aster">
+<robot xmlns:xacro="http://www.ros.org/wiki/xacro">
     <ros2_control name="RobotSystem" type="system">
         <xacro:property name="PI" value="3.14159265359" />
@@ -105,5 +105,5 @@
             <command_interface name="position">
                 <param name="min">0.0</param>
-                <param name="max">${PI/2}</param>
+                <param name="max">${PI / 2}</param>
             </command_interface>
             <state_interface name="position" />
