Commit message: in work

File: aster_description/urdf/aster.urdf.xacro (robot description, xacro)
@@ -3,7 +3,5 @@
     <xacro:include filename="$(find aster_description)/urdf/material.xacro"/>
     <xacro:include filename="$(find aster_description)/urdf/aster.xacro"/>
-<!--
-    <xacro:include filename="$(find aster_description)/urdf/aster_gazebo.xacro"/>
-    <xacro:include filename="$(find aster_description)/urdf/aster_ros2_control.xacro"/>
--->
+    <xacro:include filename="$(find aster_description)/urdf/gazebo.xacro"/>
+    <xacro:include filename="$(find aster_description)/urdf/ros2_control.xacro"/>
 </robot>

File: aster_description/urdf/aster.xacro (robot description, xacro)
@@ -7,5 +7,5 @@
             <plugin>transmission_interface/SimpleTransmission</plugin>
             <actuator name="motor_${number}" role="actuator1"/>
-            <joint name="joint_${number}"    role="joint1">
+            <joint name="joint_${number}" role="joint1">
                 <mechanical_reduction>1.0</mechanical_reduction>
             </joint>
@@ -240,5 +240,5 @@
         <xacro:default_inertial mass="0.3"/>
     </link>
-    <!-- Right Gripper-->
+    <!-- Right Gripper
     <link name="rh_rotate_top_link" >
         <visual>
@@ -320,6 +320,6 @@
         </collision>
         <xacro:default_inertial_1 mass="0.03"/>
-    </link>
-    <!-- Left Arm-->
+    </link> -->
+    <!-- Left Arm
     <link name="shoulder_lh_link">
         <visual>
@@ -401,6 +401,6 @@
         </collision>
         <xacro:default_inertial mass="0.3"/>
-    </link>
-    <!-- Left Gripper-->
+    </link> -->
+    <!-- Left Gripper
     <link name="lh_rotate_top_link" >
         <visual>
@@ -482,6 +482,6 @@
         </collision>
         <xacro:default_inertial mass="0.3"/>
-    </link>
-    <!-- Right Leg-->
+    </link> -->
+    <!-- Right Leg
     <link name="hip_rh_link">
         <visual>
@@ -531,6 +531,6 @@
         </collision>
         <xacro:default_inertial mass="0.3"/>
-    </link>
-    <!-- Left Leg-->
+    </link> -->
+    <!-- Left Leg
     <link name="hip_lh_link">
         <visual>
@@ -580,5 +580,5 @@
         </collision>
         <xacro:default_inertial mass="0.3"/>
-    </link>
+    </link> -->
                     <!-- ######  JOINTS  ######-->
     <!-- Base Virtual Joints-->
@@ -669,5 +669,5 @@
         <origin xyz="0 -0.01 -0.13" rpy="0 0 0"/>
     </joint>
-    <!-- Right Gripper Joints-->
+    <!-- Right Gripper Joints
     <joint name="gripper_body_rh" type="fixed">
         <parent link="rh_rotate_link"/>
@@ -699,6 +699,6 @@
         <child link="rh_gripper2_pad_link"/>
         <origin xyz="0 -0.015 -0.041" rpy="0.0 0.0 0.0"/>
-    </joint>
-    <!-- Left Arm Joints-->
+    </joint>  -->
+    <!-- Left Arm Joints
     <joint name="joint_9" type="revolute">
         <parent link="chest_link"/>
@@ -735,6 +735,6 @@
         <limit lower="${-PI/2}" upper="0" velocity="50.0" effort="1000.0"/>
         <origin xyz="0 0.015 -0.13" rpy="0 0 0"/>
-    </joint>
-    <!-- Left Gripper Joints-->
+    </joint> -->
+    <!-- Left Gripper Joints
     <joint name="gripper_body_lh" type="fixed">
         <parent link="lh_rotate_link"/>
@@ -766,6 +766,6 @@
         <child link="lh_gripper2_pad_link"/>
         <origin xyz="0 -0.015 -0.041" rpy="0.0 0.0 0.0"/>
-    </joint>
-    <!-- Right Leg Joints-->
+    </joint> -->
+    <!-- Right Leg Joints
     <joint name="joint_15" type="revolute">
         <parent link="hip_link"/>
@@ -788,6 +788,6 @@
         <limit lower="${-PI/4}" upper="${PI/4}" velocity="50.0" effort="1000.0"/>
         <origin xyz="0 0 -0.18" rpy="0 0 0"/>
-    </joint>
-    <!-- Left Leg Joints-->
+    </joint> -->
+    <!-- Left Leg Joints
     <joint name="joint_18" type="revolute">
         <parent link="hip_link"/>
@@ -810,25 +810,25 @@
         <limit lower="${-PI/4}" upper="${PI/4}" velocity="50.0" effort="1000.0"/>
         <origin xyz="0 0 -0.18" rpy="0 0 0"/>
-    </joint>
+    </joint>    -->
     <!-- Transmissions-->
-    <xacro:default_transmission number="1"/>
+    <xacro:default_transmission number="1"/> <!-- Head-->
     <xacro:default_transmission number="2"/>
-    <xacro:default_transmission number="3"/>
+    <xacro:default_transmission number="3"/> <!-- Right Arm-->
     <xacro:default_transmission number="4"/>
     <xacro:default_transmission number="5"/>
     <xacro:default_transmission number="6"/>
     <xacro:default_transmission number="7"/>
-    <xacro:default_transmission number="8"/>
-    <xacro:default_transmission number="9"/>
+<!--    <xacro:default_transmission number="8"/>  Right Gripper -->
+<!--    <xacro:default_transmission number="9"/>  Left Arm
     <xacro:default_transmission number="10"/>
     <xacro:default_transmission number="11"/>
     <xacro:default_transmission number="12"/>
-    <xacro:default_transmission number="13"/>
-    <xacro:default_transmission number="14"/>
-    <xacro:default_transmission number="15"/>
+    <xacro:default_transmission number="13"/> -->
+<!--    <xacro:default_transmission number="14"/>  Left Gripper -->
+<!--    <xacro:default_transmission number="15"/>  Right Leg
     <xacro:default_transmission number="16"/>
-    <xacro:default_transmission number="17"/>
-    <xacro:default_transmission number="18"/>
+    <xacro:default_transmission number="17"/> -->
+<!--    <xacro:default_transmission number="18"/>  Left Leg
     <xacro:default_transmission number="19"/>
-    <xacro:default_transmission number="20"/>
+    <xacro:default_transmission number="20"/> -->
 </robot>

File: aster_description/urdf/gazebo.xacro (robot description, xacro)
@@ -1,4 +1,4 @@
 <?xml version="1.0"?>
-<robot xmlns:xacro="http://www.ros.org/wiki/xacro" name="aster" >
+<robot xmlns:xacro="http://www.ros.org/wiki/xacro" name="aster">
     <!-- Gazebo ros2_control plugin -->
     <gazebo>
@@ -6,6 +6,7 @@
         <robot_param>robot_description</robot_param>
         <robot_param_node>robot_state_publisher</robot_param_node>
-        <parameters>$(find aster_controller)/config/aster_controllers.yaml</parameters>
+        <parameters></parameters>
       </plugin>
     </gazebo>
+<!-- $(find aster_controller)/config/aster_controllers.yaml -->
 </robot>
