Commit message: in work

File: aster_description/urdf/aster.urdf.xacro (robot description, xacro)
@@ -4,4 +4,6 @@
     <xacro:include filename="$(find aster_description)/urdf/aster.xacro"/>
     <xacro:include filename="$(find aster_description)/urdf/gazebo.xacro"/>
+<!--
     <xacro:include filename="$(find aster_description)/urdf/ros2_control.xacro"/>
+-->
 </robot>

File: aster_description/urdf/aster.xacro (robot description, xacro)
@@ -270,371 +270,415 @@
         <xacro:default_inertial mass="0.3" />
     </link>
-    <!-- Right Gripper
-    <link name="rh_rotate_top_link" >
-        <visual>
-            <origin xyz="-0.004 0.0 -0.03" rpy="${-PI/2} 0.0 ${-PI/2}"/>
-            <geometry>
-                <mesh filename="package://aster_description/meshes/Greifer/files/Robotic_Arm_Palm_Top.stl"
-    scale="0.001 0.001 0.001"/>
-            </geometry>
-            <material name="white"/>
-        </visual>
-        <collision>
-            <origin xyz="-0.004 0.0 -0.03" rpy="${-PI/2} 0.0 ${-PI/2}"/>
-            <geometry>
-                <mesh filename="package://aster_description/meshes/Greifer/files/Robotic_Arm_Palm_Top.stl"
-    scale="0.001 0.001 0.001"/>
-            </geometry>
-        </collision>
-        <xacro:default_inertial mass="0.3"/>
-    </link>
-    <link name="rh_gripper1_link" >
-        <visual>
-            <origin xyz="-0.005 0.016 -0.008" rpy="${-PI/2} 0.0 ${-PI/2}"/>
-            <geometry>
-                <mesh filename="package://aster_description/meshes/Greifer/files/Robotic_Arm_Finger.stl"
-    scale="0.001 0.001 0.001"/>
-            </geometry>
-            <material name="white"/>
-        </visual>
-        <collision>
-            <origin xyz="-0.005 0.016 -0.008" rpy="${-PI/2} 0.0 ${-PI/2}"/>
-            <geometry>
-                <mesh filename="package://aster_description/meshes/Greifer/files/Robotic_Arm_Finger.stl"
-    scale="0.001 0.001 0.001"/>
-            </geometry>
-        </collision>
-        <xacro:default_inertial mass="0.3"/>
-    </link>
-    <link name="rh_gripper2_link" >
-        <visual>
-            <origin xyz="0.007 -0.016 -0.008" rpy="${-PI/2} 0.0 ${PI/2}"/>
-            <geometry>
-                <mesh filename="package://aster_description/meshes/Greifer/files/Robotic_Arm_Finger.stl"
-    scale="0.001 0.001 0.001"/>
-            </geometry>
-            <material name="white"/>
-        </visual>
-        <collision>
-            <origin xyz="0.007 -0.016 -0.008" rpy="${-PI/2} 0.0 ${PI/2}"/>
-            <geometry>
-                <mesh filename="package://aster_description/meshes/Greifer/files/Robotic_Arm_Finger.stl"
-    scale="0.001 0.001 0.001"/>
-            </geometry>
-        </collision>
-        <xacro:default_inertial mass="0.3"/>
-    </link>
-    <link name="rh_gripper1_pad_link" >
-        <visual>
-            <origin xyz="-0.004 -0.0015 -0.0017" rpy="0.0 ${PI/2} 0.0"/>
-            <geometry>
-                <mesh filename="package://aster_description/meshes/Greifer/files/Robotic_Arm_Finger_Pad.stl"
-    scale="0.001 0.001 0.001"/>
-            </geometry>
-            <material name="black"/>
-        </visual>
-        <collision>
-            <origin xyz="-0.004 -0.0015 -0.0017" rpy="0.0 ${PI/2} 0.0"/>
-            <geometry>
-                <mesh filename="package://aster_description/meshes/Greifer/files/Robotic_Arm_Finger_Pad.stl"
-    scale="0.001 0.001 0.001"/>
-            </geometry>
-        </collision>
-        <xacro:default_inertial_1 mass="0.03"/>
-    </link>
-    <link name="rh_gripper2_pad_link" >
-        <visual>
-            <origin xyz="0.005 0.0015 -0.0017" rpy="${PI} ${PI/2} 0.0"/>
-            <geometry>
-                <mesh filename="package://aster_description/meshes/Greifer/files/Robotic_Arm_Finger_Pad.stl"
-    scale="0.001 0.001 0.001"/>
-            </geometry>
-            <material name="black"/>
-        </visual>
-        <collision>
-            <origin xyz="0.005 0.0015 -0.0017" rpy="${PI} ${PI/2} 0.0"/>
-            <geometry>
-                <mesh filename="package://aster_description/meshes/Greifer/files/Robotic_Arm_Finger_Pad.stl"
-    scale="0.001 0.001 0.001"/>
-            </geometry>
-        </collision>
-        <xacro:default_inertial_1 mass="0.03"/>
-    </link> -->
-    <!-- Left Arm
+    <!-- Right Gripper -->
+    <link name="rh_rotate_top_link">
+        <visual>
+            <origin xyz="-0.004 0.0 -0.03" rpy="${-PI/2} 0.0 ${-PI/2}" />
+            <geometry>
+                <mesh
+                    filename="package://aster_description/meshes/Greifer/files/Robotic_Arm_Palm_Top.stl"
+                    scale="0.001 0.001 0.001" />
+            </geometry>
+            <material name="white" />
+        </visual>
+        <collision>
+            <origin xyz="-0.004 0.0 -0.03" rpy="${-PI/2} 0.0 ${-PI/2}" />
+            <geometry>
+                <mesh
+                    filename="package://aster_description/meshes/Greifer/files/Robotic_Arm_Palm_Top.stl"
+                    scale="0.001 0.001 0.001" />
+            </geometry>
+        </collision>
+        <xacro:default_inertial mass="0.3" />
+    </link>
+    <link name="rh_gripper1_link">
+        <visual>
+            <origin xyz="-0.005 0.016 -0.008" rpy="${-PI/2} 0.0 ${-PI/2}" />
+            <geometry>
+                <mesh
+                    filename="package://aster_description/meshes/Greifer/files/Robotic_Arm_Finger.stl"
+                    scale="0.001 0.001 0.001" />
+            </geometry>
+            <material name="white" />
+        </visual>
+        <collision>
+            <origin xyz="-0.005 0.016 -0.008" rpy="${-PI/2} 0.0 ${-PI/2}" />
+            <geometry>
+                <mesh
+                    filename="package://aster_description/meshes/Greifer/files/Robotic_Arm_Finger.stl"
+                    scale="0.001 0.001 0.001" />
+            </geometry>
+        </collision>
+        <xacro:default_inertial mass="0.3" />
+    </link>
+    <link name="rh_gripper2_link">
+        <visual>
+            <origin xyz="0.007 -0.016 -0.008" rpy="${-PI/2} 0.0 ${PI/2}" />
+            <geometry>
+                <mesh
+                    filename="package://aster_description/meshes/Greifer/files/Robotic_Arm_Finger.stl"
+                    scale="0.001 0.001 0.001" />
+            </geometry>
+            <material name="white" />
+        </visual>
+        <collision>
+            <origin xyz="0.007 -0.016 -0.008" rpy="${-PI/2} 0.0 ${PI/2}" />
+            <geometry>
+                <mesh
+                    filename="package://aster_description/meshes/Greifer/files/Robotic_Arm_Finger.stl"
+                    scale="0.001 0.001 0.001" />
+            </geometry>
+        </collision>
+        <xacro:default_inertial mass="0.3" />
+    </link>
+    <link name="rh_gripper1_pad_link">
+        <visual>
+            <origin xyz="-0.004 -0.0015 -0.0017" rpy="0.0 ${PI/2} 0.0" />
+            <geometry>
+                <mesh
+                    filename="package://aster_description/meshes/Greifer/files/Robotic_Arm_Finger_Pad.stl"
+                    scale="0.001 0.001 0.001" />
+            </geometry>
+            <material name="black" />
+        </visual>
+        <collision>
+            <origin xyz="-0.004 -0.0015 -0.0017" rpy="0.0 ${PI/2} 0.0" />
+            <geometry>
+                <mesh
+                    filename="package://aster_description/meshes/Greifer/files/Robotic_Arm_Finger_Pad.stl"
+                    scale="0.001 0.001 0.001" />
+            </geometry>
+        </collision>
+        <xacro:default_inertial_1 gewicht="0.03" />
+    </link>
+    <link name="rh_gripper2_pad_link">
+        <visual>
+            <origin xyz="0.005 0.0015 -0.0017" rpy="${PI} ${PI/2} 0.0" />
+            <geometry>
+                <mesh
+                    filename="package://aster_description/meshes/Greifer/files/Robotic_Arm_Finger_Pad.stl"
+                    scale="0.001 0.001 0.001" />
+            </geometry>
+            <material name="black" />
+        </visual>
+        <collision>
+            <origin xyz="0.005 0.0015 -0.0017" rpy="${PI} ${PI/2} 0.0" />
+            <geometry>
+                <mesh
+                    filename="package://aster_description/meshes/Greifer/files/Robotic_Arm_Finger_Pad.stl"
+                    scale="0.001 0.001 0.001" />
+            </geometry>
+        </collision>
+        <xacro:default_inertial_1 gewicht="0.03" />
+    </link>
+    <!-- Left Arm -->
     <link name="shoulder_lh_link">
         <visual>
-            <origin xyz="-0.01 0.018 -0.023" rpy="0.0 0.0 0.0"/>
-            <geometry>
-                <mesh filename="package://aster_description/meshes/Left_Arm_Shoulder_Connector.stl" scale="0.001
-    0.001 0.001"/>
-            </geometry>
-            <material name="white"/>
-        </visual>
-        <collision>
-            <origin xyz="-0.01 0.018 -0.023" rpy="0.0 0.0 0.0"/>
-            <geometry>
-                <mesh filename="package://aster_description/meshes/Left_Arm_Shoulder_Connector.stl" scale="0.001
-    0.001 0.001"/>
-            </geometry>
-        </collision>
-        <xacro:default_inertial mass="0.3"/>
+            <origin xyz="-0.01 0.018 -0.023" rpy="0.0 0.0 0.0" />
+            <geometry>
+                <mesh filename="package://aster_description/meshes/Left_Arm_Shoulder_Connector.stl"
+                    scale="0.001
+    0.001 0.001" />
+            </geometry>
+            <material name="white" />
+        </visual>
+        <collision>
+            <origin xyz="-0.01 0.018 -0.023" rpy="0.0 0.0 0.0" />
+            <geometry>
+                <mesh filename="package://aster_description/meshes/Left_Arm_Shoulder_Connector.stl"
+                    scale="0.001
+    0.001 0.001" />
+            </geometry>
+        </collision>
+        <xacro:default_inertial mass="0.3" />
     </link>
     <link name="sh_lh_lift_link">
         <visual>
-            <origin xyz="0.0 0.0 -0.036" rpy="0.0 0.0 0.0"/>
-            <geometry>
-                <mesh filename="package://aster_description/meshes/Left_Arm_Shoulder.stl" scale="0.001 0.001
-    0.001"/>
-            </geometry>
-            <material name="white"/>
-        </visual>
-        <collision>
-            <origin xyz="0.0 0.0 -0.036" rpy="0.0 0.0 0.0"/>
-            <geometry>
-                <mesh filename="package://aster_description/meshes/Left_Arm_Shoulder.stl" scale="0.001 0.001
-    0.001"/>
-            </geometry>
-        </collision>
-        <xacro:default_inertial mass="0.3"/>
+            <origin xyz="0.0 0.0 -0.036" rpy="0.0 0.0 0.0" />
+            <geometry>
+                <mesh filename="package://aster_description/meshes/Left_Arm_Shoulder.stl"
+                    scale="0.001 0.001
+    0.001" />
+            </geometry>
+            <material name="white" />
+        </visual>
+        <collision>
+            <origin xyz="0.0 0.0 -0.036" rpy="0.0 0.0 0.0" />
+            <geometry>
+                <mesh filename="package://aster_description/meshes/Left_Arm_Shoulder.stl"
+                    scale="0.001 0.001
+    0.001" />
+            </geometry>
+        </collision>
+        <xacro:default_inertial mass="0.3" />
     </link>
     <link name="sh_lh_rotate_link">
         <visual>
-            <origin xyz="0.0 0.0 -0.005" rpy="${PI} 0.0 ${PI}"/>
-            <geometry>
-                <mesh filename="package://aster_description/meshes/Left_Arm_Upper.stl" scale="0.001 0.001 0.001"/>
-            </geometry>
-            <material name="white"/>
-        </visual>
-        <collision>
-            <origin xyz="0.0 0.0 -0.005" rpy="${PI} 0.0 ${PI}"/>
-            <geometry>
-                <mesh filename="package://aster_description/meshes/Left_Arm_Upper.stl" scale="0.001 0.001 0.001"/>
-            </geometry>
-        </collision>
-        <xacro:default_inertial mass="0.3"/>
+            <origin xyz="0.0 0.0 -0.005" rpy="${PI} 0.0 ${PI}" />
+            <geometry>
+                <mesh filename="package://aster_description/meshes/Left_Arm_Upper.stl"
+                    scale="0.001 0.001 0.001" />
+            </geometry>
+            <material name="white" />
+        </visual>
+        <collision>
+            <origin xyz="0.0 0.0 -0.005" rpy="${PI} 0.0 ${PI}" />
+            <geometry>
+                <mesh filename="package://aster_description/meshes/Left_Arm_Upper.stl"
+                    scale="0.001 0.001 0.001" />
+            </geometry>
+        </collision>
+        <xacro:default_inertial mass="0.3" />
     </link>
     <link name="elbow_lh_link">
         <visual>
-            <origin xyz="-0.06 0.002 -0.008" rpy="0.0 0.0 0.0"/>
-            <geometry>
-                <mesh filename="package://aster_description/meshes/Left_Arm_Lower.stl" scale="0.001 0.001 0.001"/>
-            </geometry>
-            <material name="white"/>
-        </visual>
-        <collision>
-            <origin xyz="-0.06 0.002 -0.008" rpy="0.0 0.0 0.0"/>
-            <geometry>
-                <mesh filename="package://aster_description/meshes/Left_Arm_Lower.stl" scale="0.001 0.001 0.001"/>
-            </geometry>
-        </collision>
-        <xacro:default_inertial mass="0.3"/>
-    </link>
-    <link name="lh_rotate_link" >
-        <visual>
-            <origin xyz="-0.02 0.0 -0.03" rpy="${-PI/2} 0.0 ${-PI/2}"/>
-            <geometry>
-                <mesh filename="package://aster_description/meshes/Greifer/files/Robotic_Arm_Palm.stl" scale="0.001
-    0.001 0.001"/>
-            </geometry>
-            <material name="white"/>
-        </visual>
-        <collision>
-            <origin xyz="-0.02 0.0 -0.03" rpy="${-PI/2} 0.0 ${-PI/2}"/>
-            <geometry>
-                <mesh filename="package://aster_description/meshes/Greifer/files/Robotic_Arm_Palm.stl" scale="0.001
-    0.001 0.001"/>
-            </geometry>
-        </collision>
-        <xacro:default_inertial mass="0.3"/>
-    </link> -->
-    <!-- Left Gripper
-    <link name="lh_rotate_top_link" >
-        <visual>
-            <origin xyz="-0.004 0.0 -0.03" rpy="${-PI/2} 0.0 ${-PI/2}"/>
-            <geometry>
-                <mesh filename="package://aster_description/meshes/Greifer/files/Robotic_Arm_Palm_Top.stl"
-    scale="0.001 0.001 0.001"/>
-            </geometry>
-            <material name="white"/>
-        </visual>
-        <collision>
-            <origin xyz="-0.004 0.0 -0.03" rpy="${-PI/2} 0.0 ${-PI/2}"/>
-            <geometry>
-                <mesh filename="package://aster_description/meshes/Greifer/files/Robotic_Arm_Palm_Top.stl"
-    scale="0.001 0.001 0.001"/>
-            </geometry>
-        </collision>
-        <xacro:default_inertial mass="0.3"/>
-    </link>
-    <link name="lh_gripper1_link" >
-        <visual>
-            <origin xyz="-0.005 0.016 -0.008" rpy="${-PI/2} 0.0 ${-PI/2}"/>
-            <geometry>
-                <mesh filename="package://aster_description/meshes/Greifer/files/Robotic_Arm_Finger.stl"
-    scale="0.001 0.001 0.001"/>
-            </geometry>
-            <material name="white"/>
-        </visual>
-        <collision>
-            <origin xyz="-0.005 0.016 -0.008" rpy="${-PI/2} 0.0 ${-PI/2}"/>
-            <geometry>
-                <mesh filename="package://aster_description/meshes/Greifer/files/Robotic_Arm_Finger.stl"
-    scale="0.001 0.001 0.001"/>
-            </geometry>
-        </collision>
-        <xacro:default_inertial mass="0.3"/>
-    </link>
-    <link name="lh_gripper2_link" >
-        <visual>
-            <origin xyz="0.007 -0.016 -0.008" rpy="${-PI/2} 0.0 ${PI/2}"/>
-            <geometry>
-                <mesh filename="package://aster_description/meshes/Greifer/files/Robotic_Arm_Finger.stl"
-    scale="0.001 0.001 0.001"/>
-            </geometry>
-            <material name="white"/>
-        </visual>
-        <collision>
-            <origin xyz="0.007 -0.016 -0.008" rpy="${-PI/2} 0.0 ${PI/2}"/>
-            <geometry>
-                <mesh filename="package://aster_description/meshes/Greifer/files/Robotic_Arm_Finger.stl"
-    scale="0.001 0.001 0.001"/>
-            </geometry>
-        </collision>
-        <xacro:default_inertial mass="0.3"/>
-    </link>
-    <link name="lh_gripper1_pad_link" >
-        <visual>
-            <origin xyz="-0.004 -0.0015 -0.0017" rpy="0.0 ${PI/2} 0.0"/>
-            <geometry>
-                <mesh filename="package://aster_description/meshes/Greifer/files/Robotic_Arm_Finger_Pad.stl"
-    scale="0.001 0.001 0.001"/>
-            </geometry>
-            <material name="black"/>
-        </visual>
-        <collision>
-            <origin xyz="-0.004 -0.0015 -0.0017" rpy="0.0 ${PI/2} 0.0"/>
-            <geometry>
-                <mesh filename="package://aster_description/meshes/Greifer/files/Robotic_Arm_Finger_Pad.stl"
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
File: aster_description/urdf/gazebo.xacro (robot description, xacro)
@@ -1,4 +1,5 @@
 <?xml version="1.0"?>
-<robot xmlns:xacro="http://www.ros.org/wiki/xacro" name="rca">
+<robot xmlns:xacro="http://www.ros.org/wiki/xacro" name="aster">
+<!--
     <gazebo>
         <plugin filename="libgazebo_ros2_control.so" name="gazebo_ros2_control">
@@ -8,5 +9,5 @@
         </plugin>
     </gazebo>
-<!--
+ -->
     <gazebo reference="base_link">
         <material>Gazebo/Black</material>
@@ -36,4 +37,3 @@
         <material>Gazebo/Black</material>
     </gazebo>
-    -->
 </robot>

File: aster_description/urdf/material.xacro (robot description, xacro)
@@ -22,7 +22,7 @@
         </inertial>
     </xacro:macro>
-    <xacro:macro name="default_inertial_1" params="masse"> <!-- <xacro:default_inertial_1 mass="1.0"/> -->
+    <xacro:macro name="default_inertial_1" params="gewicht"> <!-- <xacro:default_inertial_1 mass="1.0"/> -->
         <inertial>
-            <mass value="${masse}" />
+            <mass value="${gewicht}" />
             <inertia ixx="0.00001" ixy="0.0" ixz="0.0"
                 iyy="0.00001" iyz="0.0"
