Commit message: added camera in gazebo

File: aster_description/urdf/aster.urdf.xacro (robot description, xacro)
@@ -4,4 +4,5 @@
     <xacro:include filename="$(find aster_description)/urdf/aster.xacro"/>
     <xacro:include filename="$(find aster_description)/urdf/gazebo.xacro"/>
+    <xacro:include filename="$(find aster_description)/urdf/camera.xacro"/>
 <!--
     <xacro:include filename="$(find aster_description)/urdf/ros2_control.xacro"/>

File: aster_description/urdf/aster.xacro (robot description, xacro)
@@ -2,5 +2,5 @@
 <robot xmlns:xacro="http://www.ros.org/wiki/xacro" name="aster">
     <!-- <xacro:default_inertial mass="0.3"/> -->
-    <!-- <xacro:default_inertial_1 mass="0.03"/> -->
+    <!-- <xacro:default_inertial_1 gewicht="0.03"/> -->
     <xacro:macro name="default_transmission" params="number">
         <transmission name="transmission_${number}">

File: aster_description/urdf/gazebo.xacro (robot description, xacro)
@@ -1,5 +1,4 @@
 <?xml version="1.0"?>
 <robot xmlns:xacro="http://www.ros.org/wiki/xacro" name="aster">
-<!--
     <gazebo>
         <plugin filename="libgazebo_ros2_control.so" name="gazebo_ros2_control">
@@ -9,5 +8,4 @@
         </plugin>
     </gazebo>
- -->
     <gazebo reference="base_link">
         <material>Gazebo/Black</material>
@@ -20,5 +18,5 @@
     </gazebo>
     <gazebo reference="chest_link">
-        <material>Gazebo/White</material>
+        <material>Gazebo/Black</material>
     </gazebo>
     <gazebo reference="backbone_link">
@@ -37,3 +35,81 @@
         <material>Gazebo/Black</material>
     </gazebo>
+    <gazebo reference="shoulder_rh_link">
+        <material>Gazebo/White</material>
+    </gazebo>
+    <gazebo reference="sh_rh_lift_link">
+        <material>Gazebo/White</material>
+    </gazebo>
+    <gazebo reference="sh_rh_rotate_link">
+        <material>Gazebo/White</material>
+    </gazebo>
+    <gazebo reference="elbow_rh_link">
+        <material>Gazebo/White</material>
+    </gazebo>
+    <gazebo reference="rh_rotate_link">
+        <material>Gazebo/White</material>
+    </gazebo>
+    <gazebo reference="rh_rotate_top_link">
+        <material>Gazebo/White</material>
+    </gazebo>
+    <gazebo reference="rh_gripper1_link">
+        <material>Gazebo/White</material>
+    </gazebo>
+    <gazebo reference="rh_gripper2_link">
+        <material>Gazebo/White</material>
+    </gazebo>
+    <gazebo reference="rh_gripper1_pad_link">
+        <material>Gazebo/Blue</material>
+    </gazebo>
+    <gazebo reference="rh_gripper2_pad_link">
+        <material>Gazebo/Blue</material>
+    </gazebo>
+    <gazebo reference="shoulder_lh_link">
+        <material>Gazebo/White</material>
+    </gazebo>
+    <gazebo reference="sh_lh_lift_link">
+        <material>Gazebo/White</material>
+    </gazebo>
+    <gazebo reference="sh_lh_rotate_link">
+        <material>Gazebo/White</material>
+    </gazebo>
+    <gazebo reference="elbow_lh_link">
+        <material>Gazebo/White</material>
+    </gazebo>
+    <gazebo reference="lh_rotate_link">
+        <material>Gazebo/White</material>
+    </gazebo>
+    <gazebo reference="lh_rotate_top_link">
+        <material>Gazebo/White</material>
+    </gazebo>
+    <gazebo reference="lh_gripper1_link">
+        <material>Gazebo/White</material>
+    </gazebo>
+    <gazebo reference="lh_gripper2_link">
+        <material>Gazebo/White</material>
+    </gazebo>
+    <gazebo reference="lh_gripper1_pad_link">
+        <material>Gazebo/Blue</material>
+    </gazebo>
+    <gazebo reference="lh_gripper2_pad_link">
+        <material>Gazebo/Blue</material>
+    </gazebo>
+    <gazebo reference="hip_rh_link">
+        <material>Gazebo/White</material>
+    </gazebo>
+    <gazebo reference="knie_rh_link">
+        <material>Gazebo/White</material>
+    </gazebo>
+    <gazebo reference="foot_rh_link">
+        <material>Gazebo/Black</material>
+    </gazebo>
+    <gazebo reference="hip_lh_link">
+        <material>Gazebo/White</material>
+    </gazebo>
+    <gazebo reference="knie_lh_link">
+        <material>Gazebo/White</material>
+    </gazebo>
+    <gazebo reference="foot_lh_link">
+        <material>Gazebo/Black</material>
+    </gazebo>
 </robot>

File: aster_description/urdf/material.xacro (robot description, xacro)
@@ -30,3 +30,29 @@
         </inertial>
     </xacro:macro>
+    <xacro:macro name="box_inertia" params="m l w h xyz rpy">
+        <inertial>
+            <origin xyz="${xyz}" rpy="${rpy}" />
+            <mass value="${m}" />
+            <inertia ixx="${(m/12) * (h*h + l*l)}" ixy="0" ixz="0"
+                     iyy="${(m/12) * (w*w + l*l)}" iyz="0"
+                     izz="${(m/12) * (w*w + h*h)}" />
+        </inertial>
+    </xacro:macro>
+    <!--
+        <xacro:box_inertia m="" l="" w="" h=""
+                           xyz="0 0 0" rpy="0 0 0"/>
+    -->
+    <xacro:macro name="cylinder_inertia" params="m r h xyz rpy">
+        <inertial>
+            <origin xyz="${xyz}" rpy="${rpy}" />
+            <mass value="${m}" />
+            <inertia ixx="${(m/12) * (3*r*r + h*h)}" ixy="0" ixz="0"
+                     iyy="${(m/12) * (3*r*r + h*h)}" iyz="0"
+                     izz="${(m/2) * (r*r)}" />
+        </inertial>
+    </xacro:macro>
+    <!--
+        <xacro:cylinder_inertia m="" r="" h=""
+                           xyz="0 0 0" rpy="0 0 0"/>
+    -->
 </robot>
